File: RT08-ProgramBoard.kicad_sch (KiCad schematic)
At the start: 138 parts, among them J1 PWR/Addr, J2 PWR/Ctrl, J3 Instruction, J4 Data, J5 Instruction, J6 Data

Commit message: Schematics with 'sub-schematics' almost done
Connections:
- net Rst is gone; now on net SRAM-cell/Rst: J1.3 (Pin_3)
- net WE0 is gone; now on net D7: PQ15.2 (C)
- net D0: now reaches J3.1 (Pin_1)
- net D0: now also R9.2; no longer R16.2
- net D3: now reaches R12.2
- net D3: now also J3.4 (Pin_4); no longer J3.5 (Pin_5)
- net D1: now reaches J3.2 (Pin_2)
- net D1: now also R10.2; no longer R15.2
- net D7: now reaches J3.8 (Pin_8)
- net D7: now also R16.2; no longer R9.2
- net D14: now reaches J4.7 (Pin_7)
- net D14: now also R23.2; no longer R18.2
- net D4: now reaches R13.2
- net D4: now also J3.5 (Pin_5); no longer J3.4 (Pin_4)
- net D11: now reaches R20.2
- net D11: now also J4.4 (Pin_4); no longer J4.5 (Pin_5)
- net D2: now reaches J3.3 (Pin_3)
- net D2: now also R11.2; no longer R14.2
- net D5: now reaches J3.6 (Pin_6)
- net D5: now also R14.2; no longer R11.2
- net D6: now reaches J3.7 (Pin_7)
- net D6: now also R15.2; no longer R10.2
- net D15: now reaches R24.2
- net D15: now also J4.8 (Pin_8); no longer J4.1 (Pin_1)
- net D9: now reaches J4.2 (Pin_2)
- net D9: now also R18.2; no longer R23.2
- net D10: now reaches J4.3 (Pin_3)
- net D10: now also R19.2; no longer R22.2
- net D12: now reaches R21.2
- net D12: now also J4.5 (Pin_5); no longer J4.4 (Pin_4)
- net D13: now reaches J4.6 (Pin_6)
- net D13: now also R22.2; no longer R19.2
- net D8: now reaches R17.2
- net D8: now also J4.1 (Pin_1); no longer J4.8 (Pin_8)
Other:
- moved on the sheet: BD1, BD2, BD3, BD4, BD5, BD6, D1, D10, D11, D12, D13, D14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

Commit message: Finished editing .sch
Connections:
- net D7: no longer PQ15.2 (C)
- net P0: now reaches J5.1 (Pin_1)
- net P1: now reaches J5.2 (Pin_2)
- net P2: now reaches J5.3 (Pin_3)
- net P3: now reaches J5.4 (Pin_4)
- net P4: now reaches J5.5 (Pin_5)
- net P5: now reaches J5.6 (Pin_6)
- net P6: now reaches J5.7 (Pin_7)
- net P7: now reaches J5.8 (Pin_8)
- net P8: now reaches J6.1 (Pin_1)
- net P9: now reaches J6.2 (Pin_2)
- net P10: now reaches J6.3 (Pin_3)
- net P11: now reaches J6.4 (Pin_4)
- net P12: now reaches J6.5 (Pin_5)
- net P13: now reaches J6.6 (Pin_6)
- net P14: now reaches J6.7 (Pin_7)
- net P15: now reaches J6.8 (Pin_8)
- net SRAM-cell111/Rst renamed SRAM-cell0/Rst
- new net WE0: PQ15.2 (C)
Other:
- sheet SRAM-cell renamed SRAM-cell111
- added sheet SRAM-cell0 (Cell.kicad_sch)
- added sheet SRAM-cell1 (Cell.kicad_sch)
- added sheet SRAM-cell10 (Cell.kicad_sch)
- added sheet SRAM-cell100 (Cell.kicad_sch)
- added sheet SRAM-cell101 (Cell.kicad_sch)
- added sheet SRAM-cell102 (Cell.kicad_sch)
- added sheet SRAM-cell103 (Cell.kicad_sch)
- added sheet SRAM-cell104 (Cell.kicad_sch)
- added sheet SRAM-cell105 (Cell.kicad_sch)
- added sheet SRAM-cell106 (Cell.kicad_sch)
- added sheet SRAM-cell107 (Cell.kicad_sch)
- added sheet SRAM-cell108 (Cell.kicad_sch)
- added sheet SRAM-cell109 (Cell.kicad_sch)
- added sheet SRAM-cell11 (Cell.kicad_sch)
- added sheet SRAM-cell110 (Cell.kicad_sch)
- added sheet SRAM-cell112 (Cell.kicad_sch)
- added sheet SRAM-cell113 (Cell.kicad_sch)
- added sheet SRAM-cell114 (Cell.kicad_sch)
- added sheet SRAM-cell115 (Cell.kicad_sch)
- added sheet SRAM-cell116 (Cell.kicad_sch)
- added sheet SRAM-cell117 (Cell.kicad_sch)
- added sheet SRAM-cell118 (Cell.kicad_sch)
- added sheet SRAM-cell119 (Cell.kicad_sch)
- added sheet SRAM-cell12 (Cell.kicad_sch)
- added sheet SRAM-cell120 (Cell.kicad_sch)
- added sheet SRAM-cell121 (Cell.kicad_sch)
- added sheet SRAM-cell122 (Cell.kicad_sch)
- added sheet SRAM-cell123 (Cell.kicad_sch)
- added sheet SRAM-cell124 (Cell.kicad_sch)
- added sheet SRAM-cell125 (Cell.kicad_sch)
- added sheet SRAM-cell126 (Cell.kicad_sch)
- added sheet SRAM-cell127 (Cell.kicad_sch)
- added sheet SRAM-cell13 (Cell.kicad_sch)
- added sheet SRAM-cell14 (Cell.kicad_sch)
- added sheet SRAM-cell15 (Cell.kicad_sch)
- added sheet SRAM-cell16 (Cell.kicad_sch)
- added sheet SRAM-cell17 (Cell.kicad_sch)
- added sheet SRAM-cell18 (Cell.kicad_sch)
- added sheet SRAM-cell19 (Cell.kicad_sch)
- added sheet SRAM-cell2 (Cell.kicad_sch)
- added sheet SRAM-cell20 (Cell.kicad_sch)
- added sheet SRAM-cell21 (Cell.kicad_sch)
- added sheet SRAM-cell22 (Cell.kicad_sch)
- added sheet SRAM-cell23 (Cell.kicad_sch)
- added sheet SRAM-cell24 (Cell.kicad_sch)
- added sheet SRAM-cell25 (Cell.kicad_sch)
- added sheet SRAM-cell26 (Cell.kicad_sch)
- added sheet SRAM-cell27 (Cell.kicad_sch)
- added sheet SRAM-cell28 (Cell.kicad_sch)
- added sheet SRAM-cell29 (Cell.kicad_sch)
- added sheet SRAM-cell3 (Cell.kicad_sch)
- added sheet SRAM-cell30 (Cell.kicad_sch)
- added sheet SRAM-cell31 (Cell.kicad_sch)
- added sheet SRAM-cell32 (Cell.kicad_sch)
- added sheet SRAM-cell33 (Cell.kicad_sch)
- added sheet SRAM-cell34 (Cell.kicad_sch)
- added sheet SRAM-cell35 (Cell.kicad_sch)
- added sheet SRAM-cell36 (Cell.kicad_sch)
- added sheet SRAM-cell37 (Cell.kicad_sch)
- added sheet SRAM-cell38 (Cell.kicad_sch)
- added sheet SRAM-cell39 (Cell.kicad_sch)
- added sheet SRAM-cell4 (Cell.kicad_sch)
- added sheet SRAM-cell40 (Cell.kicad_sch)
- added sheet SRAM-cell41 (Cell.kicad_sch)
- added sheet SRAM-cell42 (Cell.kicad_sch)
- added sheet SRAM-cell43 (Cell.kicad_sch)
- added sheet SRAM-cell44 (Cell.kicad_sch)
- added sheet SRAM-cell45 (Cell.kicad_sch)
- added sheet SRAM-cell46 (Cell.kicad_sch)
- added sheet SRAM-cell47 (Cell.kicad_sch)
- added sheet SRAM-cell48 (Cell.kicad_sch)
- added sheet SRAM-cell49 (Cell.kicad_sch)
- added sheet SRAM-cell5 (Cell.kicad_sch)
- added sheet SRAM-cell50 (Cell.kicad_sch)
- added sheet SRAM-cell51 (Cell.kicad_sch)
- added sheet SRAM-cell52 (Cell.kicad_sch)
- added sheet SRAM-cell53 (Cell.kicad_sch)
- added sheet SRAM-cell54 (Cell.kicad_sch)
- added sheet SRAM-cell55 (Cell.kicad_sch)
- added sheet SRAM-cell56 (Cell.kicad_sch)
- added sheet SRAM-cell57 (Cell.kicad_sch)
- added sheet SRAM-cell58 (Cell.kicad_sch)
- added sheet SRAM-cell59 (Cell.kicad_sch)
- added sheet SRAM-cell6 (Cell.kicad_sch)
- added sheet SRAM-cell60 (Cell.kicad_sch)
- added sheet SRAM-cell61 (Cell.kicad_sch)
- added sheet SRAM-cell62 (Cell.kicad_sch)
- added sheet SRAM-cell63 (Cell.kicad_sch)
- added sheet SRAM-cell64 (Cell.kicad_sch)
- added sheet SRAM-cell65 (Cell.kicad_sch)
- added sheet SRAM-cell66 (Cell.kicad_sch)
- added sheet SRAM-cell67 (Cell.kicad_sch)
- added sheet SRAM-cell68 (Cell.kicad_sch)
- added sheet SRAM-cell69 (Cell.kicad_sch)
- added sheet SRAM-cell7 (Cell.kicad_sch)
- added sheet SRAM-cell70 (Cell.kicad_sch)
- added sheet SRAM-cell71 (Cell.kicad_sch)
- added sheet SRAM-cell72 (Cell.kicad_sch)
- added sheet SRAM-cell73 (Cell.kicad_sch)
- added sheet SRAM-cell74 (Cell.kicad_sch)
- added sheet SRAM-cell75 (Cell.kicad_sch)
- added sheet SRAM-cell76 (Cell.kicad_sch)
- added sheet SRAM-cell77 (Cell.kicad_sch)
- added sheet SRAM-cell78 (Cell.kicad_sch)
- added sheet SRAM-cell79 (Cell.kicad_sch)
- added sheet SRAM-cell8 (Cell.kicad_sch)
- added sheet SRAM-cell80 (Cell.kicad_sch)
- added sheet SRAM-cell81 (Cell.kicad_sch)
- added sheet SRAM-cell82 (Cell.kicad_sch)
- added sheet SRAM-cell83 (Cell.kicad_sch)
- added sheet SRAM-cell84 (Cell.kicad_sch)
- added sheet SRAM-cell85 (Cell.kicad_sch)
- added sheet SRAM-cell86 (Cell.kicad_sch)
- added sheet SRAM-cell87 (Cell.kicad_sch)
- added sheet SRAM-cell88 (Cell.kicad_sch)
- added sheet SRAM-cell89 (Cell.kicad_sch)
- added sheet SRAM-cell9 (Cell.kicad_sch)
- added sheet SRAM-cell90 (Cell.kicad_sch)
- added sheet SRAM-cell91 (Cell.kicad_sch)
- added sheet SRAM-cell92 (Cell.kicad_sch)
- added sheet SRAM-cell93 (Cell.kicad_sch)
- added sheet SRAM-cell94 (Cell.kicad_sch)
- added sheet SRAM-cell95 (Cell.kicad_sch)
- added sheet SRAM-cell96 (Cell.kicad_sch)
- added sheet SRAM-cell97 (Cell.kicad_sch)
- added sheet SRAM-cell98 (Cell.kicad_sch)
- added sheet SRAM-cell99 (Cell.kicad_sch)
- moved on the sheet: J5, J6

Commit message: Editing PCB, 1 cell temp-done
Connections:
- net G is gone; now on net GND: D1.1 (K), D10.1 (K), D11.1 (K), D12.1 (K), D13.1 (K), D14.1 (K), D15.1 (K), D16.1 (K), D2.1 (K), D3.1 (K), D4.1 (K), D5.1 (K), D6.1 (K), D7.1 (K), D8.1 (K), D9.1 (K), NQ19.1 (E), NQ22.1 (E), NQ25.1 (E), NQ28.1 (E), NQ31.1 (E), NQ34.1 (E), NQ37.1 (E), NQ40.1 (E), NQ43.1 (E), NQ46.1 (E), NQ49.1 (E), NQ52.1 (E), NQ55.1 (E), NQ58.1 (E), NQ61.1 (E), NQ64.1 (E)
Changed lines of the file:
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@@
 			)
 		)
-		(property "Value" "G"
+		(property "Value" "GND"
 			(at 526.542 61.468 0)
 			(effects
@@
 			)
 		)
-		(property "Value" "G"
+		(property "Value" "GND"
 			(at 374.142 61.468 0)
 			(effects
@@
 			)
 		)
-		(property "Value" "G"
+		(property "Value" "GND"
 			(at 297.942 86.868 0)
 			(effects
@@
 			)
 		)
-		(property "Value" "G"
+		(property "Value" "GND"
 			(at 336.042 61.468 0)
 			(effects
@@
 			)
 		)
-		(property "Value" "G"
+		(property "Value" "GND"
 			(at 450.342 61.468 0)
 			(effects
@@
 			)
 		)
-		(property "Value" "G"
-			(at 44.704 142.494 0)
+		(property "Value" "GND"
+			(at 45.72 147.32 0)
 			(effects
 				(font
@@
 			)
 		)
-		(property "Value" "G"
+		(property "Value" "GND"
 			(at 450.342 86.868 0)
 			(effects
@@
 			)
 		)
-		(property "Value" "G"
+		(property "Value" "GND"
 			(at 526.542 86.868 0)
 			(effects
@@
 			)
 		)
-		(property "Value" "G"
+		(property "Value" "GND"
 			(at 336.042 86.868 0)
 			(effects
@@
 			)
 		)
-		(property "Value" "G"
+		(property "Value" "GND"
 			(at 412.242 86.868 0)
 			(effects
@@
 			)
 		)
-		(property "Value" "G"
+		(property "Value" "GND"
 			(at 488.442 86.868 0)
 			(effects
@@
 			)
 		)
-		(property "Value" "G"
+		(property "Value" "GND"
 			(at 564.642 61.468 0)
 			(effects
@@
 			)
 		)
-		(property "Value" "G"
+		(property "Value" "GND"
 			(at 412.242 61.468 0)
 			(effects
@@
 			)
 		)
-		(property "Value" "G"
+		(property "Value" "GND"
 			(at 374.142 86.868 0)
 			(effects
@@
 			)
 		)
-		(property "Value" "G"
+		(property "Value" "GND"
 			(at 488.442 61.468 0)
 			(effects
@@
 			)
 		)
-		(property "Value" "G"
+		(property "Value" "GND"
 			(at 297.942 61.468 0)
 			(effects
@@
 			)
 		)
-		(property "Value" "G"
+		(property "Value" "GND"
 			(at 564.642 86.868 0)
 			(effects

Commit message: Edited title n' stuff
Other:
- company: @yoshi-jp -> @7654jp
Changed lines of the file:
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@@
 	(title_block
 		(title "Y-tran RT-08 Program board")
-		(date "2025~")
+		(date "2025/3~5")
 		(rev "B")
-		(company "@yoshi-jp")
+		(company "@7654jp")
 		(comment 2 "to provide instructions.")
 		(comment 3 "the core via 'Program base'")
