File: RT08-ProgramBoard.kicad_sch (KiCad schematic)
At the start: 138 parts, among them J1 PWR/Addr, J2 PWR/Ctrl, J3 Instruction, J4 Data, J5 Instruction, J6 Data

Commit message: Adding buffer to Rst signal
Connections:
- net SRAM-cell0/Rst renamed Rst
Other:
- added sheet Buffer0 (buf.kicad_sch)
- added sheet Buffer1 (buf.kicad_sch)
- added sheet Buffer2 (buf.kicad_sch)
- added sheet Buffer3 (buf.kicad_sch)

Commit message: Edited Sch, changed buffer from daisy chain to get from root
Other:
- added sheet Buffer4 (buf.kicad_sch)
- added sheet Buffer5 (buf.kicad_sch)
- added sheet Buffer6 (buf.kicad_sch)
- added sheet Buffer7 (buf.kicad_sch)

Commit message: Changing from 8x16 to 4x16, size issue
Parts:
- removed BD1, BD2: 30V1A, Diode_THT:D_DO-35_SOD27_P7.62mm_Horizontal, symbol Device:D_Schottky_Small_Filled
- removed J2: PWR/Ctrl, Connector_PinHeader_2.54mm:PinHeader_1x06_P2.54mm_Horizontal, symbol Connector:Conn_01x06_Pin
- removed NQ1, NQ17, NQ18, NQ19, NQ2, NQ20, NQ21, NQ22, NQ23, NQ24, NQ25, NQ26, NQ27, NQ28, NQ29, NQ30, NQ31, NQ32, NQ33, NQ34, NQ35, NQ36, NQ37, NQ38, NQ39, NQ40, NQ41, NQ42, NQ43, NQ44, NQ45, NQ46, NQ47, NQ48, NQ49, NQ50, NQ51, NQ52, NQ53, NQ54, NQ55, NQ56, NQ57, NQ58, NQ59, NQ60, NQ61, NQ62, NQ63, NQ64: DTC114E-THT, Package_TO_SOT_THT:TO-92_Inline, symbol YoshLibrary:DTC114E-THT
- removed NQ10, NQ11, NQ12, NQ13, NQ14, NQ15, NQ16, NQ7, NQ8, NQ9: DTC143E-THT, Package_TO_SOT_THT:TO-92_Inline, symbol YoshLibrary:DTC143E-THT
- removed PQ1, PQ10, PQ11, PQ12, PQ13, PQ14, PQ15, PQ16, PQ17, PQ18, PQ19, PQ2, PQ20, PQ21, PQ22, PQ3, PQ4, PQ5, PQ6, PQ7, PQ8, PQ9: DTA143E-THT, Package_TO_SOT_THT:TO-92_Inline, symbol YoshLibrary:DTA143E-THT
- removed R1, R4, R5, R6, R7, R8: 5.1k, Resistor_THT:R_Axial_DIN0207_L6.3mm_D2.5mm_P7.62mm_Horizontal, symbol Device:R_Small
- J4: value Data -> Instruction
Connections:
- net M0 is gone; now on net H0: NQ4.2 (C), R2.2
- net M1 is gone; now on net H1: NQ3.1 (E)
- net D0: now also J3.8 (Pin_8); no longer J3.1 (Pin_1)
- net D1: now also J3.7 (Pin_7); no longer J3.2 (Pin_2)
- net D10: now also J4.6 (Pin_6); no longer J4.3 (Pin_3)
- net D11: now also J4.5 (Pin_5); no longer J4.4 (Pin_4)
- net D12: now also J4.4 (Pin_4); no longer J4.5 (Pin_5)
- net D13: now also J4.3 (Pin_3); no longer J4.6 (Pin_6)
- net D14: now also J4.2 (Pin_2); no longer J4.7 (Pin_7)
- net D15: now also J4.1 (Pin_1); no longer J4.8 (Pin_8)
- net D2: now also J3.6 (Pin_6); no longer J3.3 (Pin_3)
- net D3: now also J3.5 (Pin_5); no longer J3.4 (Pin_4)
- net D4: now also J3.4 (Pin_4); no longer J3.5 (Pin_5)
- net D5: now also J3.3 (Pin_3); no longer J3.6 (Pin_6)
- net D6: now also J3.2 (Pin_2); no longer J3.7 (Pin_7)
- net D7: now also J3.1 (Pin_1); no longer J3.8 (Pin_8)
- net D8: now also J4.8 (Pin_8); no longer J4.1 (Pin_1)
- net D9: now also J4.7 (Pin_7); no longer J4.2 (Pin_2)
- net DataEn: now also J1.4 (Pin_4)
- net GND: no longer J1.7 (Pin_7)
- net P0: now also J5.8 (Pin_8); no longer J5.1 (Pin_1)
- net P1: now also J5.7 (Pin_7); no longer J5.2 (Pin_2)
- net P10: now also J6.6 (Pin_6); no longer J6.3 (Pin_3)
- net P11: now also J6.5 (Pin_5); no longer J6.4 (Pin_4)
- net P12: now also J6.4 (Pin_4); no longer J6.5 (Pin_5)
- net P13: now also J6.3 (Pin_3); no longer J6.6 (Pin_6)
- net P14: now also J6.2 (Pin_2); no longer J6.7 (Pin_7)
- net P15: now also J6.1 (Pin_1); no longer J6.8 (Pin_8)
- net P2: now also J5.6 (Pin_6); no longer J5.3 (Pin_3)
- net P3: now also J5.5 (Pin_5); no longer J5.4 (Pin_4)
- net P4: now also J5.4 (Pin_4); no longer J5.5 (Pin_5)
- net P5: now also J5.3 (Pin_3); no longer J5.6 (Pin_6)
- net P6: now also J5.2 (Pin_2); no longer J5.7 (Pin_7)
- net P7: now also J5.1 (Pin_1); no longer J5.8 (Pin_8)
- net P8: now also J6.8 (Pin_8); no longer J6.1 (Pin_1)
- net P9: now also J6.7 (Pin_7); no longer J6.2 (Pin_2)
- net Rst: now also J1.5 (Pin_5); no longer J1.3 (Pin_3)
- net WriteEn: now also J1.3 (Pin_3)
- net Addr13: no longer names the net of J1.6 (Pin_6)
- net Addr13: now also NQ5.3 (B), NQ6.3 (B)
- net Addr14: no longer names the net of NQ3.3 (B), NQ4.3 (B)
- net Addr14: now also J1.7 (Pin_7); no longer J1.5 (Pin_5)
- removed net Addr15: J1.4 (Pin_4), NQ5.3 (B), NQ6.3 (B)
Other:
- removed sheet Buffer4
- removed sheet Buffer5
- removed sheet Buffer6
- removed sheet Buffer7
- removed sheet SRAM-cell100
- removed sheet SRAM-cell101
- removed sheet SRAM-cell102
- removed sheet SRAM-cell103
- removed sheet SRAM-cell104
- removed sheet SRAM-cell105
- removed sheet SRAM-cell106
- removed sheet SRAM-cell107
- removed sheet SRAM-cell108
- removed sheet SRAM-cell109
- removed sheet SRAM-cell110
- removed sheet SRAM-cell111
- removed sheet SRAM-cell112
- removed sheet SRAM-cell113
- removed sheet SRAM-cell114
- removed sheet SRAM-cell115
- removed sheet SRAM-cell116
- removed sheet SRAM-cell117
- removed sheet SRAM-cell118
- removed sheet SRAM-cell119
- removed sheet SRAM-cell120
- removed sheet SRAM-cell121
- removed sheet SRAM-cell122
- removed sheet SRAM-cell123
- removed sheet SRAM-cell124
- removed sheet SRAM-cell125
- removed sheet SRAM-cell126
- removed sheet SRAM-cell127
- removed sheet SRAM-cell64
- removed sheet SRAM-cell65
- removed sheet SRAM-cell66
- removed sheet SRAM-cell67
- removed sheet SRAM-cell68
- removed sheet SRAM-cell69
- removed sheet SRAM-cell70
- removed sheet SRAM-cell71
- removed sheet SRAM-cell72
- removed sheet SRAM-cell73
- removed sheet SRAM-cell74
- removed sheet SRAM-cell75
- removed sheet SRAM-cell76
- removed sheet SRAM-cell77
- removed sheet SRAM-cell78
- removed sheet SRAM-cell79
- removed sheet SRAM-cell80
- removed sheet SRAM-cell81
- removed sheet SRAM-cell82
- removed sheet SRAM-cell83
- removed sheet SRAM-cell84
- removed sheet SRAM-cell85
- removed sheet SRAM-cell86
- removed sheet SRAM-cell87
- removed sheet SRAM-cell88
- removed sheet SRAM-cell89
- removed sheet SRAM-cell90
- removed sheet SRAM-cell91
- removed sheet SRAM-cell92
- removed sheet SRAM-cell93
- removed sheet SRAM-cell94
- removed sheet SRAM-cell95
- removed sheet SRAM-cell96
- removed sheet SRAM-cell97
- removed sheet SRAM-cell98
- removed sheet SRAM-cell99
- note added: "Program SRAM board 4 instructions 8 bytes"
- note added: "VDD Addr14 Addr15 Rst DEn WEn GND VDD"
- note removed: "Program SRAM board 8 instructions 16 bytes"
- note removed: "VDD GND Addr13 Addr14 Addr15 Rst GND VDD"
- note removed: "VDD GND DEn WEn GND VND"
- moved on the sheet: BD3, BD4, BD5, BD6, J1, J5, NQ3, NQ4, NQ5, NQ6, R2, R3

Commit message: Updated sch, re-create pcb next
Parts:
- removed D1, D10, D11, D12, D13, D14, D15, D16, D2, D3, D4, D5, D6, D7, D8, D9: 30V0.2A, Diode_THT:D_DO-35_SOD27_P7.62mm_Horizontal, symbol Device:D_Schottky_Small_Filled
- removed R10, R11, R12, R13, R14, R15, R16, R17, R18, R19, R20, R21, R22, R23, R24, R9: 10k, Resistor_THT:R_Axial_DIN0207_L6.3mm_D2.5mm_P7.62mm_Horizontal, symbol Device:R_Small
- added NQ10, NQ11, NQ12, NQ13, NQ14, NQ15, NQ16, NQ17, NQ18, NQ19, NQ20, NQ21, NQ22, NQ23, NQ24, NQ5, NQ6, NQ7, NQ8, NQ9: DTC114E-THT, Package_TO_SOT_THT:TO-92_Inline, symbol YoshLibrary:DTC114E-THT
- added NX1, NX2, NX3, NX4: 2SC1815, Package_TO_SOT_THT:TO-92_Inline, symbol YoshLibrary:2SC1815
- added PQ1, PQ10, PQ11, PQ12, PQ2, PQ3, PQ4, PQ5, PQ6, PQ7, PQ8, PQ9: DTA114E-THT, Package_TO_SOT_THT:TO-92_Inline, symbol YoshLibrary:DTA114E-THT
- R1: renamed from R2; value 5.1k -> 10k; footprint Resistor_THT:R_Axial_DIN0207_L6.3mm_D2.5mm_P7.62mm_Horizontal -> YoshLibrary:R_Axial_DIN0207_L6.3mm_D2.5mm_P7.62mm_Horizontal
- R2: renamed from R3; value 5.1k -> 10k; footprint Resistor_THT:R_Axial_DIN0207_L6.3mm_D2.5mm_P7.62mm_Horizontal -> YoshLibrary:R_Axial_DIN0207_L6.3mm_D2.5mm_P7.62mm_Horizontal
- renumbered BD3 to BD1, BD4 to BD2, BD5 to BD3, BD6 to BD4, J3 to J2, J4 to J3, J5 to J4, J6 to J5, NQ3 to NQ1, NQ4 to NQ2, NQ5 to NQ3, NQ6 to NQ4
Connections:
- net +5V: now also PQ1.1 (E), PQ10.1 (E), PQ11.1 (E), PQ12.1 (E), PQ2.1 (E), PQ3.1 (E), PQ4.1 (E), PQ5.1 (E), PQ6.1 (E), PQ7.1 (E), PQ8.1 (E), PQ9.1 (E)
- net DE0: now also PQ5.2 (C)
- net DE1: now also PQ6.2 (C)
- net DE2: now also PQ7.2 (C)
- net DE3: now also PQ8.2 (C)
- net DataEn: now also NQ10.3 (B), NQ12.3 (B), NQ14.3 (B), NQ16.3 (B)
- net GND: now also NQ10.1 (E), NQ12.1 (E), NQ14.1 (E), NQ16.1 (E), NQ18.1 (E), NQ20.1 (E), NQ22.1 (E), NQ24.1 (E), NQ5.1 (E), NQ6.1 (E), NQ8.1 (E), NX2.1 (E)
- net H0: now also NX1.3 (B), NX3.3 (B)
- net H1: now also NQ7.3 (B), NX4.3 (B)
- net L0: now also NQ6.3 (B), NX2.3 (B)
- net L1: now also NQ5.3 (B), NQ8.3 (B)
- net WE0: now also PQ9.2 (C)
- net WE1: now also PQ10.2 (C)
- net WE2: now also PQ11.2 (C)
- net WE3: now also PQ12.2 (C)
- net WriteEn: now also NQ18.3 (B), NQ20.3 (B), NQ22.3 (B), NQ24.3 (B)
- new net: NQ19.1 (E), NQ20.2 (C)
- new net: NQ15.2 (C), PQ8.3 (B)
- new net: NX1.1 (E), NX2.2 (C)
- new net: NX1.2 (C), PQ1.3 (B)
- new net: NQ21.1 (E), NQ22.2 (C)
- new net: NQ11.1 (E), NQ12.2 (C)
- new net: NQ11.2 (C), PQ6.3 (B)
- new net: NQ9.2 (C), PQ5.3 (B)
- new net: NQ7.2 (C), PQ4.3 (B)
- new net: NQ7.1 (E), NQ8.2 (C)
- new net: NQ21.2 (C), PQ11.3 (B)
- new net: NQ19.2 (C), PQ10.3 (B)
- new net: NQ6.2 (C), NX4.1 (E)
- new net: NX4.2 (C), PQ3.3 (B)
- new net: NQ17.1 (E), NQ18.2 (C)
- new net: NQ17.2 (C), PQ9.3 (B)
- new net: NQ23.2 (C), PQ12.3 (B)
- new net: NQ15.1 (E), NQ16.2 (C)
- new net: NQ13.1 (E), NQ14.2 (C)
- new net: NQ23.1 (E), NQ24.2 (C)
- new net: NQ10.2 (C), NQ9.1 (E)
- new net: NQ5.2 (C), NX3.1 (E)
- new net: NX3.2 (C), PQ2.3 (B)
- new net: NQ13.2 (C), PQ7.3 (B)
- new net S0: NQ17.3 (B), NQ9.3 (B), PQ1.2 (C)
- new net S1: NQ11.3 (B), NQ19.3 (B), PQ2.2 (C)
- new net S2: NQ13.3 (B), NQ21.3 (B), PQ3.2 (C)
- new net S3: NQ15.3 (B), NQ23.3 (B), PQ4.2 (C)
Other:
- moved on the sheet: J2, J3

Commit message: Editing PCB, 2to4 encoder temp-done
Connections:
- net GND: now also NX4.1 (E); no longer NQ6.1 (E)
- net H1: now also NQ6.3 (B); no longer NX4.3 (B)
- net L0: now also NX4.3 (B); no longer NQ6.3 (B)
- net at NQ6.2 (C): now also PQ3.3 (B); no longer NX4.1 (E)
- net at NX4.2 (C): now also NQ6.1 (E); no longer PQ3.3 (B)
Other:
- moved on the sheet: NQ6, NX4
Changed lines of the file:
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@@
 	(symbol
 		(lib_id "YoshLibrary:2SC1815")
-		(at 176.53 81.28 0)
+		(at 186.69 82.55 0)
 		(unit 1)
 		(exclude_from_sim no)
@@
 		(dnp no)
 		(property "Reference" "NX4"
-			(at 171.45 76.835 0)
+			(at 181.61 78.74 0)
 			(effects
 				(font
@@
 		)
 		(property "Value" "2SC1815"
-			(at 181.61 82.5499 0)
+			(at 191.77 83.8199 0)
 			(effects
 				(font
@@
 		)
 		(property "Footprint" "Package_TO_SOT_THT:TO-92_Inline"
-			(at 181.61 83.185 0)
+			(at 191.77 84.455 0)
 			(effects
 				(font
@@
 		)
 		(property "Datasheet" "https://media.digikey.com/pdf/Data%20Sheets/Toshiba%20PDFs/2SC1815.pdf"
-			(at 176.53 81.28 0)
+			(at 186.69 82.55 0)
 			(effects
 				(font
@@
 		)
 		(property "Description" "0.15A Ic, 50V Vce, Low Noise Audio NPN Transistor, TO-92"
-			(at 176.53 81.28 0)
+			(at 186.69 82.55 0)
 			(effects
 				(font
@@
 	(symbol
 		(lib_id "YoshLibrary:DTC114E-THT")
-		(at 186.69 82.55 0)
+		(at 176.53 81.28 0)
 		(unit 1)
 		(exclude_from_sim no)
@@
 		(dnp no)
 		(property "Reference" "NQ6"
-			(at 181.61 78.74 0)
+			(at 171.45 77.47 0)
 			(effects
 				(font
@@
 		)
 		(property "Value" "DTC114E-THT"
-			(at 191.77 83.8199 0)
+			(at 181.61 82.5499 0)
 			(effects
 				(font
@@
 		)
 		(property "Footprint" "Package_TO_SOT_THT:TO-92_Inline"
-			(at 186.69 82.55 0)
-			(effects
-				(font
-					(size 1.27 1.27)
-				)
-				(justify left)
-				(hide yes)
-			)
-		)
-		(property "Datasheet" ""
-			(at 186.69 82.55 0)
+			(at 176.53 81.28 0)
+			(effects
+				(font
+					(size 1.27 1.27)
+				)
+				(justify left)
+				(hide yes)
+			)
+		)
+		(property "Datasheet" ""
+			(at 176.53 81.28 0)
 			(effects
 				(font
@@
 		)
 		(property "Description" "Digital NPN Transistor, 10k/10k, TO-92"
-			(at 186.944 87.122 0)
-			(effects
-				(font
+			(at 176.784 85.852 0)
+			(effects
+				(font

Commit message: Changed size, 1 inst per board. Updating everything
Parts:
- removed BD1, BD2, BD3, BD4: 30V1A, Diode_THT:D_DO-35_SOD27_P7.62mm_Horizontal, symbol Device:D_Schottky_Small_Filled
- removed NQ1, NQ10, NQ11, NQ12, NQ13, NQ14, NQ15, NQ16, NQ17, NQ18, NQ19, NQ2, NQ20, NQ21, NQ22, NQ23, NQ24, NQ3, NQ4, NQ5, NQ6, NQ7, NQ8, NQ9: DTC114E-THT, Package_TO_SOT_THT:TO-92_Inline, symbol YoshLibrary:DTC114E-THT
- removed NX1, NX2, NX3, NX4: 2SC1815, Package_TO_SOT_THT:TO-92_Inline, symbol YoshLibrary:2SC1815
- removed PQ1, PQ10, PQ11, PQ12, PQ2, PQ3, PQ4, PQ5, PQ6, PQ7, PQ8, PQ9: DTA114E-THT, Package_TO_SOT_THT:TO-92_Inline, symbol YoshLibrary:DTA114E-THT
- removed R1, R2: 10k, YoshLibrary:R_Axial_DIN0207_L6.3mm_D2.5mm_P7.62mm_Horizontal, symbol Device:R_Small
- J3: value Instruction -> Data
Connections:
- net GND: now also J1.5 (Pin_5), J1.7 (Pin_7)
- net Rst: now also J1.6 (Pin_6); no longer J1.5 (Pin_5)
- net DataEn renamed DEn
- net WriteEn renamed WEn
Other:
- removed sheet Buffer0
- removed sheet Buffer1
- removed sheet Buffer2
- removed sheet Buffer3
- removed sheet SRAM-cell16
- removed sheet SRAM-cell17
- removed sheet SRAM-cell18
- removed sheet SRAM-cell19
- removed sheet SRAM-cell20
- removed sheet SRAM-cell21
- removed sheet SRAM-cell22
- removed sheet SRAM-cell23
- removed sheet SRAM-cell24
- removed sheet SRAM-cell25
- removed sheet SRAM-cell26
- removed sheet SRAM-cell27
- removed sheet SRAM-cell28
- removed sheet SRAM-cell29
- removed sheet SRAM-cell30
- removed sheet SRAM-cell31
- removed sheet SRAM-cell32
- removed sheet SRAM-cell33
- removed sheet SRAM-cell34
- removed sheet SRAM-cell35
- removed sheet SRAM-cell36
- removed sheet SRAM-cell37
- removed sheet SRAM-cell38
- removed sheet SRAM-cell39
- removed sheet SRAM-cell40
- removed sheet SRAM-cell41
- removed sheet SRAM-cell42
- removed sheet SRAM-cell43
- removed sheet SRAM-cell44
- removed sheet SRAM-cell45
- removed sheet SRAM-cell46
- removed sheet SRAM-cell47
- removed sheet SRAM-cell48
- removed sheet SRAM-cell49
- removed sheet SRAM-cell50
- removed sheet SRAM-cell51
- removed sheet SRAM-cell52
- removed sheet SRAM-cell53
- removed sheet SRAM-cell54
- removed sheet SRAM-cell55
- removed sheet SRAM-cell56
- removed sheet SRAM-cell57
- removed sheet SRAM-cell58
- removed sheet SRAM-cell59
- removed sheet SRAM-cell60
- removed sheet SRAM-cell61
- removed sheet SRAM-cell62
- removed sheet SRAM-cell63
- note added: "Program SRAM board 1 inst.=2 bytes"
- note added: "VDD GND Rst GND DEn WEn GND VDD"
- note removed: "Program SRAM board 4 instructions 8 bytes"
- note removed: "VDD Addr14 Addr15 Rst DEn WEn GND VDD"
- moved on the sheet: J1, J2, J3, J4, J5

Commit message: Optimized for univ. board
Other:
- moved on the sheet: J1, J2, J3, J4, J5
