File: buf.kicad_sch (KiCad schematic)
At the start: 2 parts

Commit message: Updated sch, re-create pcb next
Parts:
- renumbered NQ961 to NQ25, PQ279 to PQ13
Changed lines of the file:
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@@
 		(on_board yes)
 		(dnp no)
-		(property "Reference" "#PWR0613"
+		(property "Reference" "#PWR066001"
 			(at 27.94 30.48 0)
 			(effects
@@
 			(project "RT08-ProgramBoard"
 				(path "/1e4a9b72-5dca-4cd4-9b5c-6a0bbded1998/8cb9a0e2-ac9e-4f8e-905d-48e2924bf956"
-					(reference "#PWR0613")
+					(reference "#PWR066001")
 					(unit 1)
 				)
 				(path "/1e4a9b72-5dca-4cd4-9b5c-6a0bbded1998/936d5558-9fc5-4fc7-a713-5fb79fe91b62"
-					(reference "#PWR0615")
+					(reference "#PWR068001")
 					(unit 1)
 				)
 				(path "/1e4a9b72-5dca-4cd4-9b5c-6a0bbded1998/c3bf8b9b-5e1b-4222-9f14-5fb269051932"
-					(reference "#PWR0617")
+					(reference "#PWR069001")
 					(unit 1)
 				)
 				(path "/1e4a9b72-5dca-4cd4-9b5c-6a0bbded1998/f48c2fe5-0d30-48d8-bec9-1dc8a6075678"
-					(reference "#PWR0614")
+					(reference "#PWR067001")
 					(unit 1)
 				)
@@
 		(on_board yes)
 		(dnp no)
-		(property "Reference" "PQ279"
+		(property "Reference" "PQ13"
 			(at 23.114 22.86 0)
 			(effects
@@
 			(project "RT08-ProgramBoard"
 				(path "/1e4a9b72-5dca-4cd4-9b5c-6a0bbded1998/8cb9a0e2-ac9e-4f8e-905d-48e2924bf956"
-					(reference "PQ279")
+					(reference "PQ13")
 					(unit 1)
 				)
 				(path "/1e4a9b72-5dca-4cd4-9b5c-6a0bbded1998/936d5558-9fc5-4fc7-a713-5fb79fe91b62"
-					(reference "PQ281")
+					(reference "PQ79")
 					(unit 1)
 				)
 				(path "/1e4a9b72-5dca-4cd4-9b5c-6a0bbded1998/c3bf8b9b-5e1b-4222-9f14-5fb269051932"
-					(reference "PQ283")
+					(reference "PQ112")
 					(unit 1)
 				)
 				(path "/1e4a9b72-5dca-4cd4-9b5c-6a0bbded1998/f48c2fe5-0d30-48d8-bec9-1dc8a6075678"
-					(reference "PQ280")
+					(reference "PQ46")
 					(unit 1)
 				)
@@
 		(on_board yes)
 		(dnp no)
-		(property "Reference" "NQ961"
+		(property "Reference" "NQ25"
 			(at 16.002 26.924 0)
 			(effects
@@
 			(project "RT08-ProgramBoard"
 				(path "/1e4a9b72-5dca-4cd4-9b5c-6a0bbded1998/8cb9a0e2-ac9e-4f8e-905d-48e2924bf956"
-					(reference "NQ961")
+					(reference "NQ25")
 					(unit 1)
 				)
 				(path "/1e4a9b72-5dca-4cd4-9b5c-6a0bbded1998/936d5558-9fc5-4fc7-a713-5fb79fe91b62"
-					(reference "NQ963")
+					(reference "NQ251")
 					(unit 1)
 				)
 				(path "/1e4a9b72-5dca-4cd4-9b5c-6a0bbded1998/c3bf8b9b-5e1b-4222-9f14-5fb269051932"
-					(reference "NQ965")
+					(reference "NQ364")
 					(unit 1)
 				)
 				(path "/1e4a9b72-5dca-4cd4-9b5c-6a0bbded1998/f48c2fe5-0d30-48d8-bec9-1dc8a6075678"
-					(reference "NQ962")
-					(unit 1)
-				)
+					(reference "NQ138")
+					(unit 1)
+				)
