File: RT08-ProgramBoard.kicad_pcb (KiCad board)
At the start: 2 copper layers, 384.8 x 303.5 mm, 309 parts, among them J1 PWR/Addr, J2 Instruction, J3 Data, J4 Instruction, J5 Data

Commit message: Deleted one group, ready to re-builded
Parts:
- moved C1 153.6 mm to (56.7, 214.7)
- moved D1 153.6 mm to (76.3, 211.8)
- moved D2 153.6 mm to (76.3, 215.4)
- moved NQ1 153.6 mm to (57.1, 193.0)
- moved NQ2 153.6 mm to (57.1, 198.8)
- moved NQ3 153.6 mm to (57.1, 204.6)
- moved NQ4 153.6 mm to (57.1, 210.4)
- moved NQ5 153.6 mm to (63.7, 193.0)
- moved NQ6 153.6 mm to (63.7, 198.8)
- moved NQ7 153.6 mm to (63.7, 204.6)
- moved NX1 153.6 mm to (63.7, 210.4)
- moved PQ1 153.6 mm to (70.2, 193.0)
- moved PQ2 153.6 mm to (70.2, 198.8)
- moved PX1 153.6 mm to (70.2, 204.6)
- moved R1 153.6 mm to (76.3, 191.8)
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Routing:
- net (no net): track 4791.3 -> 2105.6 mm, vias 42 -> 22
- net +5V: track 969.5 -> 436.2 mm
- net /P12: track 149.7 -> 0.00 mm, vias 1 -> 0
- net /D6: track 84.4 -> 0.00 mm, vias 1 -> 0
- net /D5: track 84.4 -> 0.00 mm, vias 1 -> 0
- net /D4: track 84.4 -> 0.00 mm, vias 1 -> 0
- net /D7: track 84.4 -> 0.00 mm, vias 1 -> 0
- net /D14: track 82.6 -> 0.00 mm
- net /D12: track 82.6 -> 0.00 mm
- net /D15: track 82.6 -> 0.00 mm
- net /D13: track 82.6 -> 0.00 mm
- net /P10: track 75.8 -> 0.00 mm, vias 1 -> 0
- net /P9: track 75.8 -> 0.00 mm, vias 1 -> 0
- net /P11: track 149.7 -> 74.0 mm, vias 1 -> 0
- net /P3: track 74.0 -> 0.00 mm
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Other:
- board size 384.8 x 303.5 mm -> 5.1 x 5.1 mm

Commit message: Optimized for univ. board
Parts:
- NQ1, NQ10, NQ100, NQ101, NQ102, NQ103, NQ104, NQ105, NQ106, NQ107, NQ108, NQ109, NQ11, NQ110, NQ111, NQ112, NQ12, NQ13, NQ14, NQ15, NQ16, NQ17, NQ18, NQ19, NQ2, NQ20, NQ21, NQ22, NQ23, NQ24, NQ25, NQ26, NQ27, NQ28, NQ29, NQ3, NQ30, NQ31, NQ32, NQ33, NQ34, NQ35, NQ36, NQ37, NQ38, NQ39, NQ4, NQ40, NQ41, NQ42, NQ43, NQ44, NQ45, NQ46, NQ47, NQ48, NQ49, NQ5, NQ50, NQ51, NQ52, NQ53, NQ54, NQ55, NQ56, NQ57, NQ58, NQ59, NQ6, NQ60, NQ61, NQ62, NQ63, NQ64, NQ65, NQ66, NQ67, NQ68, NQ69, NQ7, NQ70, NQ71, NQ72, NQ73, NQ74, NQ75, NQ76, NQ77, NQ78, NQ79, NQ8, NQ80, NQ81, NQ82, NQ83, NQ84, NQ85, NQ86, NQ87, NQ88, NQ89, NQ9, NQ90, NQ91, NQ92, NQ93, NQ94, NQ95, NQ96, NQ97, NQ98, NQ99, NX1, NX10, NX11, NX12, NX13, NX14, NX15, NX16, NX2, NX3, NX4, NX5, NX6, NX7, NX8, NX9, PQ1, PQ10, PQ11, PQ12, PQ13, PQ14, PQ15, PQ16, PQ17, PQ18, PQ19, PQ2, PQ20, PQ21, PQ22, PQ23, PQ24, PQ25, PQ26, PQ27, PQ28, PQ29, PQ3, PQ30, PQ31, PQ32, PQ4, PQ5, PQ6, PQ7, PQ8, PQ9, PX1, PX10, PX11, PX12, PX13, PX14, PX15, PX16, PX2, PX3, PX4, PX5, PX6, PX7, PX8, PX9: footprint Package_TO_SOT_THT:TO-92_Inline -> Package_TO_SOT_THT:TO-92_Inline_Wide
- moved NQ6 188.3 mm to (248.9, 165.1), turned to 180 degrees
- moved NQ7 188.1 mm to (246.4, 160.0)
- moved NX1 183.3 mm to (241.3, 165.1), turned to 180 degrees
- moved NQ4 181.6 mm to (233.7, 167.6), turned to 180 degrees
- moved PQ2 179.8 mm to (243.8, 152.4)
- moved C1 179.6 mm to (228.6, 162.6)
- moved NQ2 172.8 mm to (226.1, 162.6), turned to 180 degrees
- moved R5 171.9 mm to (241.3, 160.0), turned to 90 degrees
- moved NQ5 171.2 mm to (233.7, 172.7), turned to 180 degrees
- moved NQ3 170.5 mm to (221.0, 157.5), turned to 180 degrees
- moved PX1 169.5 mm to (233.7, 160.0)
- moved R3 166.9 mm to (236.2, 152.4), turned to 180 degrees
- moved R4 163.5 mm to (236.2, 170.2)
- moved PQ1 161.1 mm to (226.1, 152.4), turned to 180 degrees
- moved R2 159.6 mm to (231.1, 157.5), turned to 180 degrees
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Connections:
- net /DataEn renamed /DEn
- D17 pad 2: /SRAM-cell10/Rst -> /Rst
- D18 pad 2: /SRAM-cell10/Rst -> /Rst
- D19 pad 2: /SRAM-cell10/Rst -> /Rst
- D20 pad 2: /SRAM-cell10/Rst -> /Rst
- D21 pad 2: /SRAM-cell10/Rst -> /Rst
- D22 pad 2: /SRAM-cell10/Rst -> /Rst
- D23 pad 2: /SRAM-cell10/Rst -> /Rst
- D24 pad 2: /SRAM-cell10/Rst -> /Rst
- J1 pad 3: /WriteEn -> /WEn
- NQ10 pad 3: /WriteEn -> /WEn
- NQ12 pad 3: /WriteEn -> /WEn
- NQ17 pad 3: /WriteEn -> /WEn
- NQ19 pad 3: /WriteEn -> /WEn
- NQ24 pad 3: /WriteEn -> /WEn
- NQ26 pad 3: /WriteEn -> /WEn
- NQ3 pad 3: /WriteEn -> /WEn
- NQ31 pad 3: /WriteEn -> /WEn
- NQ33 pad 3: /WriteEn -> /WEn
- NQ38 pad 3: /WriteEn -> /WEn
- NQ40 pad 3: /WriteEn -> /WEn
- NQ45 pad 3: /WriteEn -> /WEn
- NQ47 pad 3: /WriteEn -> /WEn
- NQ5 pad 3: /WriteEn -> /WEn
- NQ52 pad 3: /WriteEn -> /WEn
- NQ54 pad 3: /WriteEn -> /WEn
- NQ73 pad 3: /SRAM-cell10/WE -> /WEn
- NQ74 pad 3: /SRAM-cell10/WE -> /WEn
- NQ75 pad 3: /SRAM-cell10/WE -> /WEn
- NQ76 pad 3: /SRAM-cell10/WE -> /WEn
- NQ77 pad 3: /SRAM-cell10/WE -> /WEn
- NQ78 pad 3: /SRAM-cell10/WE -> /WEn
- NQ79 pad 3: /SRAM-cell10/WE -> /WEn
- NQ80 pad 3: /SRAM-cell10/WE -> /WEn
- NQ89 pad 3: /SRAM-cell10/WE -> /WEn
- NQ90 pad 3: /SRAM-cell10/WE -> /WEn
- NQ91 pad 3: /SRAM-cell10/WE -> /WEn
- NQ92 pad 3: /SRAM-cell10/WE -> /WEn
- NQ93 pad 3: /SRAM-cell10/WE -> /WEn
- NQ94 pad 3: /SRAM-cell10/WE -> /WEn
- NQ95 pad 3: /SRAM-cell10/WE -> /WEn
- NQ96 pad 3: /SRAM-cell10/WE -> /WEn
- PQ17 pad 1: /SRAM-cell10/VDD -> +5V
- PQ18 pad 1: /SRAM-cell10/VDD -> +5V
- PQ19 pad 1: /SRAM-cell10/VDD -> +5V
- PQ20 pad 1: /SRAM-cell10/VDD -> +5V
- PQ21 pad 1: /SRAM-cell10/VDD -> +5V
- PQ22 pad 1: /SRAM-cell10/VDD -> +5V
- PQ23 pad 1: /SRAM-cell10/VDD -> +5V
- PQ24 pad 1: /SRAM-cell10/VDD -> +5V
- PQ25 pad 1: /SRAM-cell10/VDD -> +5V
- PQ26 pad 1: /SRAM-cell10/VDD -> +5V
- PQ27 pad 1: /SRAM-cell10/VDD -> +5V
- PQ28 pad 1: /SRAM-cell10/VDD -> +5V
- PQ29 pad 1: /SRAM-cell10/VDD -> +5V
- PQ30 pad 1: /SRAM-cell10/VDD -> +5V
- PQ31 pad 1: /SRAM-cell10/VDD -> +5V
- PQ32 pad 1: /SRAM-cell10/VDD -> +5V
- R1 pad 1: /WriteEn -> /WEn
- R11 pad 1: /WriteEn -> /WEn
- R16 pad 1: /WriteEn -> /WEn
- R21 pad 1: /WriteEn -> /WEn
- R26 pad 1: /WriteEn -> /WEn
- R31 pad 1: /WriteEn -> /WEn
- R36 pad 1: /WriteEn -> /WEn
- R41 pad 1: /SRAM-cell10/WE -> /WEn
- R42 pad 1: /SRAM-cell10/WE -> /WEn
- R43 pad 1: /SRAM-cell10/WE -> /WEn
- R44 pad 1: /SRAM-cell10/WE -> /WEn
- R45 pad 1: /SRAM-cell10/WE -> /WEn
- R46 pad 1: /SRAM-cell10/WE -> /WEn
- R47 pad 1: /SRAM-cell10/WE -> /WEn
- R48 pad 1: /SRAM-cell10/WE -> /WEn
- R57 pad 2: /SRAM-cell10/VDD -> +5V
- R58 pad 2: /SRAM-cell10/VDD -> +5V
- R59 pad 2: /SRAM-cell10/VDD -> +5V
- R6 pad 1: /WriteEn -> /WEn
- R60 pad 2: /SRAM-cell10/VDD -> +5V
- R61 pad 2: /SRAM-cell10/VDD -> +5V
- R62 pad 2: /SRAM-cell10/VDD -> +5V
- R63 pad 2: /SRAM-cell10/VDD -> +5V
- R64 pad 2: /SRAM-cell10/VDD -> +5V
Routing:
- net Net-(NQ4-C): track 0.00 -> 25.4 mm
- net Net-(PX1-E): track 0.00 -> 15.2 mm
- net Net-(D2-A): track 0.00 -> 15.2 mm
- net /WEn: track 0.00 -> 10.2 mm
- net Net-(NQ4-E): track 0.00 -> 7.62 mm
- net Net-(NQ2-C): track 0.00 -> 7.62 mm
- net Net-(NX1-C): track 0.00 -> 7.62 mm
- net Net-(NQ7-C): track 0.00 -> 7.62 mm
- net Net-(D1-K): track 0.00 -> 7.62 mm
- net Net-(NQ3-C): track 0.00 -> 7.62 mm
- net /D0: track 84.4 -> 89.5 mm
- net Net-(PQ1-C): track 0.00 -> 5.08 mm
- net Net-(NQ6-C): track 0.00 -> 5.08 mm
- net Net-(NQ6-B): track 0.00 -> 2.54 mm
Other:
- board outline removed

Commit message: Share footprint folder
Routing:
- net (no net): track 2105.6 -> 0.00 mm, vias 22 -> 0
- net +5V: track 436.2 -> 0.00 mm
- net /D3: track 84.4 -> 0.00 mm, vias 1 -> 0
- net /D0: track 89.5 -> 5.08 mm, vias 1 -> 0
- net /D1: track 84.4 -> 0.00 mm, vias 1 -> 0
- net /D2: track 84.4 -> 0.00 mm, vias 1 -> 0
- net /D9: track 82.6 -> 0.00 mm
- net /D11: track 82.6 -> 0.00 mm
- net /D8: track 82.6 -> 0.00 mm
- net /D10: track 82.6 -> 0.00 mm
- net /P8: track 75.8 -> 0.00 mm, vias 1 -> 0
- net /P7: track 75.8 -> 0.00 mm, vias 1 -> 0
- net /P6: track 75.8 -> 0.00 mm, vias 1 -> 0
- net /P5: track 75.8 -> 0.00 mm, vias 1 -> 0
- net /P15: track 74.0 -> 0.00 mm
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
Commit message: Assembled 4 cells, fp copied
Parts:
- moved NQ1 183.0 mm to (30.5, 172.7)
- moved R1 183.0 mm to (30.5, 160.0)
- moved C1 183.0 mm to (45.8, 170.2)
- moved D1 183.0 mm to (43.2, 180.3)
- moved D2 183.0 mm to (43.2, 177.8)
- moved NQ2 183.0 mm to (43.2, 170.2)
- moved NQ3 183.0 mm to (38.1, 165.1)
- moved NQ4 183.0 mm to (50.8, 175.3)
- moved NQ5 183.0 mm to (50.8, 180.3)
- moved NQ6 183.0 mm to (66.0, 172.7)
- moved NQ7 183.0 mm to (63.5, 167.6)
- moved NX1 183.0 mm to (58.4, 172.7)
- moved PQ1 183.0 mm to (43.2, 160.0)
- moved PQ2 183.0 mm to (61.0, 160.0)
- moved PX1 183.0 mm to (50.8, 167.6)
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Routing:
- net GND: track 0.00 -> 398.9 mm
- net +5V: track 0.00 -> 200.7 mm
- net Net-(NQ25-C): track 0.00 -> 25.4 mm
- net Net-(NQ18-C): track 0.00 -> 25.4 mm
- net Net-(NQ11-C): track 0.00 -> 25.4 mm
- net /WEn: track 10.2 -> 30.5 mm
- net Net-(D8-A): track 0.00 -> 15.2 mm
- net Net-(D6-A): track 0.00 -> 15.2 mm
- net Net-(D4-A): track 0.00 -> 15.2 mm
- net Net-(PX4-E): track 0.00 -> 15.2 mm
- net Net-(PX3-E): track 0.00 -> 15.2 mm
- net Net-(PX2-E): track 0.00 -> 15.2 mm
- net Net-(NX4-C): track 0.00 -> 7.62 mm
- net Net-(NX3-C): track 0.00 -> 7.62 mm
- net Net-(NQ25-E): track 0.00 -> 7.62 mm
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
Commit message: Did some stuff, started wiring
Parts:
- NQ102, NQ103, NQ109, NQ110, NQ60, NQ61, NQ67, NQ68, NQ74, NQ75: value DTC114E-THT -> DTC143E-THT
- NQ83, NQ84, NQ85, NQ86, NQ87, NQ90, NQ91, NQ92, NQ93, NQ94: value DTC143E-THT -> DTC114E-THT
- R43, R48, R53, R73, R78: value 5.1k -> 1k
- R44, R49, R54, R74, R79: value 5.1k -> 10k
- R57, R60, R61, R62: value 1k -> 5.1k
- R59, R64: value 1k -> 10k
- R65, R66, R67, R70, R71, R72: value 10k -> 5.1k
- R68: value 10k -> 1k
- moved R61 284.2 mm to (30.5, 259.1), turned to -90 degrees
- moved R64 268.0 mm to (53.3, 276.9), turned to 0 degrees
- moved NQ86 260.0 mm to (43.2, 269.2)
- moved NQ89 257.9 mm to (50.8, 279.4)
- moved PQ25 257.1 mm to (43.2, 259.1), turned to 180 degrees
- moved NQ92 254.2 mm to (76.2, 271.8), turned to 0 degrees
- moved R69 253.6 mm to (99.1, 276.9)
- moved NQ97 253.6 mm to (111.8, 271.8)
- moved NQ29 252.8 mm to (30.5, 205.7)
- moved R21 252.8 mm to (30.5, 193.0)
- moved R22 252.8 mm to (48.3, 198.1)
- moved C5 252.8 mm to (45.8, 203.2)
- moved D10 252.8 mm to (43.2, 210.8)
- moved D9 252.8 mm to (43.2, 213.4)
- moved NQ30 252.8 mm to (43.2, 203.2)
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Connections:
- C10 pad 2: Net-(NQ81-C) -> Net-(NQ67-C)
- C11 pad 2: Net-(NQ88-C) -> Net-(NQ74-C)
- C12 pad 2: Net-(NQ83-C) -> Net-(NQ81-C)
- C13 pad 2: Net-(NQ84-C) -> Net-(NQ88-C)
- C14 pad 2: Net-(NQ85-C) -> Net-(NQ95-C)
- C15 pad 2: Net-(NQ86-C) -> Net-(NQ102-C)
- C16 pad 2: Net-(NQ87-C) -> Net-(NQ109-C)
- C9 pad 2: Net-(NQ82-C) -> Net-(NQ60-C)
- D18 pad 1: Net-(D18-K) -> Net-(D17-K)
- D18 pad 2: /Rst -> Net-(D18-A)
- D20 pad 1: Net-(D20-K) -> Net-(D19-K)
- D20 pad 2: /Rst -> Net-(D20-A)
- D22 pad 1: Net-(D22-K) -> Net-(D21-K)
- D22 pad 2: /Rst -> Net-(D22-A)
- D24 pad 1: Net-(D24-K) -> Net-(D23-K)
- D24 pad 2: /Rst -> Net-(D24-A)
- D25 pad 1: Net-(D22-K) -> Net-(D25-K)
- D25 pad 2: Net-(D25-A) -> /Rst
- D26 pad 1: Net-(D24-K) -> Net-(D25-K)
- D27 pad 1: Net-(D18-K) -> Net-(D27-K)
- D27 pad 2: Net-(D27-A) -> /Rst
- D28 pad 1: Net-(D21-K) -> Net-(D27-K)
- D29 pad 1: Net-(D20-K) -> Net-(D29-K)
- D29 pad 2: Net-(D29-A) -> /Rst
- D30 pad 1: Net-(D23-K) -> Net-(D29-K)
- D31 pad 1: Net-(D19-K) -> Net-(D31-K)
- D31 pad 2: Net-(D31-A) -> /Rst
- D32 pad 1: Net-(D17-K) -> Net-(D31-K)
- NQ100 pad 3: Net-(NQ100-B) -> /D14
- NQ101 pad 1: GND -> Net-(NQ100-C)
- NQ101 pad 3: Net-(NQ101-B) -> /WEn
- NQ102 pad 1: GND -> Net-(NQ102-E)
- NQ102 pad 3: Net-(NQ102-B) -> Net-(D29-K)
- NQ103 pad 2: Net-(NQ103-C) -> Net-(NQ102-E)
- NQ103 pad 3: Net-(NQ103-B) -> /WEn
- NQ105 pad 1: Net-(NQ105-E) -> Net-(NQ104-C)
- NQ106 pad 1: Net-(NQ101-C) -> GND
- NQ106 pad 2: Net-(NQ106-C) -> Net-(D32-A)
- NQ106 pad 3: /SRAM-cell10/DE -> /D15
- NQ107 pad 1: Net-(NQ107-E) -> GND
- NQ107 pad 3: /SRAM-cell10/DE -> /D15
- NQ108 pad 1: Net-(NQ102-C) -> Net-(NQ107-C)
- NQ108 pad 3: /SRAM-cell10/DE -> /WEn
- NQ109 pad 3: /SRAM-cell10/DE -> Net-(D31-K)
- NQ110 pad 1: Net-(NQ104-C) -> GND
- NQ110 pad 2: Net-(NQ110-C) -> Net-(NQ109-E)
- NQ110 pad 3: /SRAM-cell10/DE -> /WEn
- NQ111 pad 1: Net-(NQ100-C) -> GND
- NQ111 pad 3: /SRAM-cell10/DE -> Net-(NQ111-B)
- NQ112 pad 1: Net-(NQ103-C) -> Net-(NQ111-C)
- NQ57 pad 2: Net-(D27-A) -> Net-(D18-A)
- NQ57 pad 3: /D12 -> /D8
- NQ58 pad 2: Net-(D32-A) -> Net-(NQ58-C)
- NQ58 pad 3: /D14 -> /D8
- NQ59 pad 1: GND -> Net-(NQ58-C)
- NQ59 pad 2: Net-(D26-A) -> Net-(NQ59-C)
- NQ59 pad 3: /D10 -> /WEn
- NQ60 pad 1: GND -> Net-(NQ60-E)
- NQ60 pad 2: Net-(D31-A) -> Net-(NQ60-C)
- NQ60 pad 3: /D15 -> Net-(D17-K)
- NQ61 pad 2: Net-(D28-A) -> Net-(NQ60-E)
- NQ61 pad 3: /D13 -> /WEn
- NQ62 pad 2: Net-(D30-A) -> Net-(NQ62-C)
- NQ62 pad 3: /D11 -> Net-(NQ62-B)
- NQ63 pad 1: GND -> Net-(NQ62-C)
- NQ63 pad 2: Net-(D25-A) -> Net-(NQ63-C)
- NQ63 pad 3: /D9 -> /SRAM-cell10/DE
- NQ64 pad 2: Net-(D29-A) -> Net-(D20-A)
- NQ64 pad 3: /D8 -> /D9
- NQ65 pad 3: /D13 -> /D9
- NQ66 pad 1: GND -> Net-(NQ65-C)
- NQ66 pad 3: /D10 -> /WEn
- NQ67 pad 1: GND -> Net-(NQ67-E)
- NQ67 pad 3: /D15 -> Net-(D19-K)
- NQ68 pad 2: Net-(NQ68-C) -> Net-(NQ67-E)
- NQ68 pad 3: /D14 -> /WEn
- NQ69 pad 3: /D12 -> Net-(NQ69-B)
- NQ70 pad 1: GND -> Net-(NQ69-C)
- NQ70 pad 3: /D9 -> /SRAM-cell10/DE
- NQ71 pad 2: Net-(NQ71-C) -> Net-(D22-A)
- NQ71 pad 3: /D8 -> /D10
- NQ72 pad 3: /D11 -> /D10
- NQ73 pad 1: Net-(NQ66-C) -> Net-(NQ72-C)
- NQ74 pad 1: Net-(NQ67-C) -> Net-(NQ74-E)
- NQ74 pad 3: /WEn -> Net-(D21-K)
- NQ75 pad 1: Net-(NQ71-C) -> GND
- NQ75 pad 2: Net-(NQ75-C) -> Net-(NQ74-E)
- NQ76 pad 1: Net-(NQ68-C) -> GND
- NQ76 pad 3: /WEn -> Net-(NQ76-B)
- NQ77 pad 1: Net-(NQ72-C) -> Net-(NQ76-C)
- NQ77 pad 3: /WEn -> /SRAM-cell10/DE
- NQ78 pad 1: Net-(NQ69-C) -> GND
- NQ78 pad 2: Net-(NQ78-C) -> Net-(D24-A)
- NQ78 pad 3: /WEn -> /D11
- NQ79 pad 1: Net-(NQ65-C) -> GND
- NQ79 pad 3: /WEn -> /D11
- NQ80 pad 1: Net-(NQ70-C) -> Net-(NQ79-C)
- NQ81 pad 3: Net-(D22-K) -> Net-(D23-K)
- NQ82 pad 1: Net-(NQ82-E) -> GND
- NQ82 pad 2: Net-(NQ82-C) -> Net-(NQ81-E)
- NQ82 pad 3: Net-(D23-K) -> /WEn
- NQ83 pad 1: Net-(NQ83-E) -> GND
- NQ83 pad 3: Net-(D17-K) -> Net-(NQ83-B)
- NQ84 pad 1: Net-(NQ84-E) -> Net-(NQ83-C)
- NQ84 pad 3: Net-(D19-K) -> /SRAM-cell10/DE
- NQ85 pad 1: Net-(NQ85-E) -> GND
- NQ85 pad 2: Net-(NQ85-C) -> Net-(D26-A)
- NQ85 pad 3: Net-(D24-K) -> /D12
- NQ86 pad 1: Net-(NQ86-E) -> GND
- NQ86 pad 3: Net-(D20-K) -> /D12
- NQ87 pad 1: Net-(NQ87-E) -> Net-(NQ86-C)
- NQ87 pad 3: Net-(D18-K) -> /WEn
- NQ88 pad 3: Net-(D21-K) -> Net-(D25-K)
- NQ89 pad 2: Net-(NQ86-E) -> Net-(NQ88-E)
- NQ90 pad 2: Net-(NQ82-E) -> Net-(NQ90-C)
- NQ90 pad 3: /WEn -> Net-(NQ90-B)
- NQ91 pad 1: GND -> Net-(NQ90-C)
- NQ91 pad 2: Net-(NQ81-E) -> Net-(NQ91-C)
- NQ91 pad 3: /WEn -> /SRAM-cell10/DE
- NQ92 pad 2: Net-(NQ83-E) -> Net-(D28-A)
- NQ92 pad 3: /WEn -> /D13
- NQ93 pad 2: Net-(NQ85-E) -> Net-(NQ93-C)
- NQ93 pad 3: /WEn -> /D13
- NQ94 pad 1: GND -> Net-(NQ93-C)
- NQ94 pad 2: Net-(NQ84-E) -> Net-(NQ94-C)
- NQ95 pad 1: GND -> Net-(NQ95-E)
- NQ95 pad 2: Net-(NQ87-E) -> Net-(NQ95-C)
- NQ95 pad 3: /WEn -> Net-(D27-K)
- NQ96 pad 2: Net-(NQ88-E) -> Net-(NQ95-E)
- NQ97 pad 2: Net-(NQ109-E) -> Net-(NQ97-C)
- NQ98 pad 1: GND -> Net-(NQ97-C)
- NQ98 pad 2: Net-(NQ105-E) -> Net-(NQ98-C)
- NQ98 pad 3: Net-(NQ98-B) -> /SRAM-cell10/DE
- NQ99 pad 2: Net-(NQ107-E) -> Net-(D30-A)
- NQ99 pad 3: Net-(NQ99-B) -> /D14
- NX10 pad 1: Net-(NQ99-B) -> Net-(NQ69-B)
- NX10 pad 3: Net-(NQ86-C) -> Net-(NQ67-C)
- NX11 pad 1: Net-(NQ97-B) -> Net-(NQ76-B)
- NX11 pad 3: Net-(NQ83-C) -> Net-(NQ74-C)
- NX12 pad 1: Net-(NQ101-B) -> Net-(NQ83-B)
- NX12 pad 3: Net-(NQ87-C) -> Net-(NQ81-C)
- NX13 pad 1: Net-(NQ98-B) -> Net-(NQ90-B)
- NX13 pad 3: Net-(NQ84-C) -> Net-(NQ88-C)
- NX14 pad 1: Net-(NQ100-B) -> Net-(NQ97-B)
- NX14 pad 3: Net-(NQ85-C) -> Net-(NQ95-C)
- NX15 pad 3: Net-(NQ81-C) -> Net-(NQ102-C)
- NX16 pad 1: Net-(NQ102-B) -> Net-(NQ111-B)
- NX16 pad 3: Net-(NQ88-C) -> Net-(NQ109-C)
- NX9 pad 1: Net-(NQ103-B) -> Net-(NQ62-B)
- NX9 pad 3: Net-(NQ82-C) -> Net-(NQ60-C)
- PQ17 pad 3: Net-(NQ73-C) -> Net-(NQ59-C)
- PQ18 pad 2: Net-(PQ18-C) -> /P8
- PQ18 pad 3: Net-(NQ77-C) -> Net-(NQ63-C)
- PQ19 pad 3: Net-(NQ80-C) -> Net-(NQ66-C)
- PQ20 pad 2: Net-(PQ20-C) -> /P9
- PQ20 pad 3: Net-(NQ78-C) -> Net-(NQ70-C)
- PQ21 pad 3: Net-(NQ76-C) -> Net-(NQ73-C)
- PQ22 pad 2: Net-(PQ22-C) -> /P10
- PQ22 pad 3: Net-(NQ74-C) -> Net-(NQ77-C)
- PQ23 pad 3: Net-(NQ75-C) -> Net-(NQ80-C)
- PQ24 pad 2: Net-(PQ24-C) -> /P11
- PQ24 pad 3: Net-(NQ79-C) -> Net-(NQ84-C)
- PQ25 pad 2: /P12 -> Net-(PQ25-C)
- PQ25 pad 3: Net-(NQ106-C) -> Net-(NQ87-C)
- PQ26 pad 2: /P11 -> /P12
- PQ26 pad 3: Net-(NQ112-C) -> Net-(NQ91-C)
- PQ27 pad 2: /P8 -> Net-(PQ27-C)
- PQ27 pad 3: Net-(NQ107-C) -> Net-(NQ94-C)
- PQ28 pad 2: /P9 -> /P13
- PQ28 pad 3: Net-(NQ110-C) -> Net-(NQ98-C)
- PQ29 pad 2: /P15 -> Net-(PQ29-C)
- PQ29 pad 3: Net-(NQ105-C) -> Net-(NQ101-C)
- PQ30 pad 3: Net-(NQ109-C) -> Net-(NQ105-C)
- PQ31 pad 2: /P10 -> Net-(PQ31-C)
- PQ31 pad 3: Net-(NQ111-C) -> Net-(NQ108-C)
- PQ32 pad 2: /P13 -> /P15
- PQ32 pad 3: Net-(NQ108-C) -> Net-(NQ112-C)
- PX10 pad 2: Net-(NQ88-C) -> Net-(NQ67-C)
- PX10 pad 3: Net-(NX16-C) -> Net-(NX10-C)
- PX11 pad 2: Net-(NQ81-C) -> Net-(NQ74-C)
- PX11 pad 3: Net-(NX15-C) -> Net-(NX11-C)
- PX12 pad 2: Net-(NQ85-C) -> Net-(NQ81-C)
- PX12 pad 3: Net-(NX14-C) -> Net-(NX12-C)
- PX13 pad 2: Net-(NQ84-C) -> Net-(NQ88-C)
- PX14 pad 2: Net-(NQ86-C) -> Net-(NQ95-C)
- PX14 pad 3: Net-(NX10-C) -> Net-(NX14-C)
- PX15 pad 2: Net-(NQ82-C) -> Net-(NQ102-C)
- PX15 pad 3: Net-(NX9-C) -> Net-(NX15-C)
- PX16 pad 2: Net-(NQ83-C) -> Net-(NQ109-C)
- PX16 pad 3: Net-(NX11-C) -> Net-(NX16-C)
- PX9 pad 2: Net-(NQ87-C) -> Net-(NQ60-C)
- PX9 pad 3: Net-(NX12-C) -> Net-(NX9-C)
- R41 pad 2: Net-(D25-A) -> Net-(D18-A)
- R42 pad 1: /WEn -> Net-(NQ60-C)
- R42 pad 2: Net-(D26-A) -> Net-(PQ17-C)
- R43 pad 1: /WEn -> Net-(PX9-E)
- R43 pad 2: Net-(D29-A) -> +5V
- R44 pad 1: /WEn -> Net-(NQ60-C)
- R44 pad 2: Net-(D30-A) -> GND
- R45 pad 1: /WEn -> Net-(NX9-C)
- R45 pad 2: Net-(D28-A) -> Net-(PX9-E)
- R46 pad 2: Net-(D31-A) -> Net-(D20-A)
- R47 pad 1: /WEn -> Net-(NQ67-C)
- R47 pad 2: Net-(D32-A) -> Net-(PQ19-C)
- R48 pad 1: /WEn -> Net-(PX10-E)
- R48 pad 2: Net-(D27-A) -> +5V
- R49 pad 1: Net-(NQ81-C) -> Net-(NQ67-C)
- R49 pad 2: Net-(PQ19-C) -> GND
- R50 pad 1: Net-(NQ85-C) -> Net-(NX10-C)
- R50 pad 2: Net-(PQ17-C) -> Net-(PX10-E)
- R51 pad 1: Net-(NQ88-C) -> /WEn
- R51 pad 2: Net-(PQ24-C) -> Net-(D22-A)
- R52 pad 1: Net-(NQ83-C) -> Net-(NQ74-C)
- R53 pad 1: Net-(NQ87-C) -> Net-(PX11-E)
- R53 pad 2: Net-(PQ20-C) -> +5V
- R54 pad 1: Net-(NQ84-C) -> Net-(NQ74-C)
- R54 pad 2: Net-(PQ22-C) -> GND
- R55 pad 1: Net-(NQ82-C) -> Net-(NX11-C)
- R55 pad 2: Net-(PQ18-C) -> Net-(PX11-E)
- R56 pad 1: Net-(NQ86-C) -> /WEn
- R56 pad 2: Net-(PQ23-C) -> Net-(D24-A)
- R57 pad 1: Net-(PX13-E) -> Net-(NQ81-C)
- R57 pad 2: +5V -> Net-(PQ23-C)
- R58 pad 1: Net-(PX15-E) -> Net-(PX12-E)
- R59 pad 1: Net-(PX14-E) -> Net-(NQ81-C)
- R59 pad 2: +5V -> GND
- R60 pad 1: Net-(PX11-E) -> Net-(NX12-C)
- R60 pad 2: +5V -> Net-(PX12-E)
- R61 pad 1: Net-(PX16-E) -> /WEn
- R61 pad 2: +5V -> Net-(D26-A)
- R62 pad 1: Net-(PX10-E) -> Net-(NQ88-C)
- R62 pad 2: +5V -> Net-(PQ25-C)
- R63 pad 1: Net-(PX12-E) -> Net-(PX13-E)
- R64 pad 1: Net-(PX9-E) -> Net-(NQ88-C)
- R64 pad 2: +5V -> GND
- R65 pad 1: Net-(NQ86-C) -> Net-(NX13-C)
- R65 pad 2: GND -> Net-(PX13-E)
- R66 pad 1: Net-(NQ82-C) -> /WEn
- R66 pad 2: GND -> Net-(D28-A)
- R67 pad 1: Net-(NQ81-C) -> Net-(NQ95-C)
- R67 pad 2: GND -> Net-(PQ27-C)
- R68 pad 1: Net-(NQ88-C) -> Net-(PX14-E)
- R68 pad 2: GND -> +5V
- R69 pad 1: Net-(NQ83-C) -> Net-(NQ95-C)
- R70 pad 1: Net-(NQ87-C) -> Net-(NX14-C)
- R70 pad 2: GND -> Net-(PX14-E)
- R71 pad 1: Net-(NQ84-C) -> /WEn
- R71 pad 2: GND -> Net-(D30-A)
- R72 pad 1: Net-(NQ85-C) -> Net-(NQ102-C)
- R72 pad 2: GND -> Net-(PQ29-C)
- R73 pad 1: Net-(NX11-C) -> Net-(PX15-E)
- R73 pad 2: Net-(PX16-E) -> +5V
- R74 pad 1: Net-(NX14-C) -> Net-(NQ102-C)
- R74 pad 2: Net-(PX12-E) -> GND
- R75 pad 1: Net-(NX12-C) -> Net-(NX15-C)
- R75 pad 2: Net-(PX9-E) -> Net-(PX15-E)
- R76 pad 1: Net-(NX16-C) -> /WEn
- R76 pad 2: Net-(PX10-E) -> Net-(D32-A)
- R77 pad 1: Net-(NX9-C) -> Net-(NQ109-C)
- R77 pad 2: Net-(PX15-E) -> Net-(PQ31-C)
- R78 pad 1: Net-(NX15-C) -> Net-(PX16-E)
- R78 pad 2: Net-(PX11-E) -> +5V
- R79 pad 1: Net-(NX10-C) -> Net-(NQ109-C)
- R79 pad 2: Net-(PX14-E) -> GND
- R80 pad 1: Net-(NX13-C) -> Net-(NX16-C)
- R80 pad 2: Net-(PX13-E) -> Net-(PX16-E)
Routing:
- net GND: track 398.9 -> 1616.1 mm
- net +5V: track 200.7 -> 843.3 mm
- net /WEn: track 30.5 -> 121.9 mm
- net Net-(NQ81-C): track 0.00 -> 25.4 mm
- net Net-(NQ74-C): track 0.00 -> 25.4 mm
- net Net-(NQ60-C): track 0.00 -> 25.4 mm
- net Net-(NQ67-C): track 0.00 -> 25.4 mm
- net Net-(NQ53-C): track 0.00 -> 25.4 mm
- net Net-(NQ46-C): track 0.00 -> 25.4 mm
- net Net-(NQ109-C): track 0.00 -> 25.4 mm
- net Net-(NQ102-C): track 0.00 -> 25.4 mm
- net Net-(NQ88-C): track 0.00 -> 25.4 mm
- net Net-(NQ32-C): track 0.00 -> 25.4 mm
- net Net-(NQ95-C): track 0.00 -> 25.4 mm
- net Net-(NQ39-C): track 0.00 -> 25.4 mm
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
Commit message: Editing Board, VDD and VCC wiring done
Parts:
- PQ1, PQ10, PQ11, PQ12, PQ13, PQ14, PQ15, PQ16, PQ17, PQ18, PQ19, PQ2, PQ20, PQ21, PQ22, PQ23, PQ24, PQ25, PQ26, PQ27, PQ28, PQ29, PQ3, PQ30, PQ31, PQ32, PQ4, PQ5, PQ6, PQ7, PQ8, PQ9: value DTA143E-THT -> DTA114E-THT
- moved C1 130.4 mm to (61.0, 40.6)
- moved C13 130.4 mm to (61.0, 139.7)
- moved C14 130.4 mm to (106.7, 139.7)
- moved C15 130.4 mm to (152.4, 139.7)
- moved C16 130.4 mm to (198.2, 139.7)
- moved C2 130.4 mm to (106.7, 40.6)
- moved C3 130.4 mm to (152.4, 40.6)
- moved C4 130.4 mm to (198.2, 40.6)
- moved D1 130.4 mm to (58.4, 50.8)
- moved D11 130.4 mm to (104.1, 83.8)
- moved D13 130.4 mm to (149.9, 83.8)
- moved D15 130.4 mm to (195.6, 83.8)
- moved D18 130.4 mm to (58.4, 114.3)
- moved D2 130.4 mm to (58.4, 48.3)
- moved D20 130.4 mm to (104.1, 114.3)
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Connections:
- J1 pad 3: /WEn -> /DEn
- J1 pad 4: /DEn -> /WEn
- NQ105 pad 3: /SRAM-cell10/DE -> /DEn
- NQ112 pad 3: /SRAM-cell10/DE -> /DEn
- NQ63 pad 3: /SRAM-cell10/DE -> /DEn
- NQ70 pad 3: /SRAM-cell10/DE -> /DEn
- NQ77 pad 3: /SRAM-cell10/DE -> /DEn
- NQ84 pad 3: /SRAM-cell10/DE -> /DEn
- NQ91 pad 3: /SRAM-cell10/DE -> /DEn
- NQ98 pad 3: /SRAM-cell10/DE -> /DEn
Routing:
- net GND: track 1616.1 -> 1626.2 mm

Commit message: Editing board, size-optimizing
Parts:
- moved C12 24.1 mm to (221.0, 99.1)
- moved NQ50 24.1 mm to (205.7, 68.6)
- moved NQ55 24.1 mm to (241.3, 68.6)
- moved NQ78 24.1 mm to (205.7, 101.6)
- moved NQ81 24.1 mm to (226.1, 104.1)
- moved NQ82 24.1 mm to (226.1, 109.2)
- moved NQ83 24.1 mm to (241.3, 101.6)
- moved NX12 24.1 mm to (233.7, 101.6)
- moved NX8 24.1 mm to (233.7, 68.6)
- moved PX12 24.1 mm to (226.1, 96.5)
- moved PX8 24.1 mm to (226.1, 63.5)
- moved R40 24.1 mm to (233.7, 63.5)
- moved R60 24.1 mm to (233.7, 96.5)
- moved C4 24.1 mm to (221.0, 33.0)
- moved C8 24.1 mm to (221.0, 66.0)
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Connections:
- J1 pad 3: /DEn -> /WEn
- J1 pad 4: /WEn -> /DEn
Routing:
- net /Rst: track 0.00 -> 160.0 mm
- net GND: track 1626.2 -> 1707.5 mm
- net +5V: track 843.3 -> 924.6 mm

Commit message: Seems done!
Parts:
- moved D32 29.3 mm to (189.2, 139.7)
- moved PX16 29.3 mm to (196.8, 129.5)
- moved R79 29.3 mm to (199.4, 139.7)
- moved R80 29.3 mm to (204.5, 129.5)
- moved C16 29.3 mm to (191.8, 132.1)
- moved D31 29.3 mm to (189.2, 142.2)
- moved NQ106 29.3 mm to (176.5, 134.6)
- moved NQ107 29.3 mm to (189.2, 132.1)
- moved NQ108 29.3 mm to (184.2, 127.0)
- moved NQ109 29.3 mm to (196.8, 137.2)
- moved NQ110 29.3 mm to (196.8, 142.2)
- moved NQ111 29.3 mm to (212.1, 134.6)
- moved NX16 29.3 mm to (204.5, 134.6)
- moved PQ31 29.3 mm to (189.2, 121.9)
- moved PQ32 29.3 mm to (207.0, 121.9)
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Routing:
- net /Rst: track 160.0 -> 0.00 mm
- net GND: track 1707.5 -> 1616.1 mm, vias 0 -> 4
- net +5V: track 924.6 -> 833.1 mm, vias 0 -> 4
- net /D7: vias 0 -> 1
- net /D3: vias 0 -> 1
- net /D15: vias 0 -> 1
- net /D11: vias 0 -> 1
- net /D9: vias 0 -> 1
- net /D5: vias 0 -> 1
- net /D13: vias 0 -> 1
- net /D1: vias 0 -> 1
- net /D8: vias 0 -> 1
- net /D4: vias 0 -> 1
- net /D12: vias 0 -> 1
- net /D0: vias 0 -> 1
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