File: RT08-ProgramBoard.kicad_pcb (KiCad board)
At the start: 2 copper layers, 190.5 x 149.9 mm, 325 parts, among them J1 PWR/Addr, J2 Inst-1, J3 Inst-2, J4 Data-1, J5 Data-2

Commit message: Remaking due to design change, wip1
Parts:
- D1, D10, D11, D12, D13, D14, D15, D16, D17, D18, D19, D2, D20, D21, D22, D23, D24, D25, D26, D27, D28, D29, D3, D30, D31, D32, D33, D34, D35, D36, D37, D38, D39, D4, D40, D41, D42, D43, D44, D45, D46, D47, D48, D5, D6, D7, D8, D9: value Schottky -> 30V0.2A
- NQ104, NQ111, NQ13, NQ20, NQ27, NQ34, NQ41, NQ48, NQ55, NQ6, NQ62, NQ69, NQ76, NQ83, NQ90, NQ97: value DTC114E-THT -> DTC143E-THT
- R1, R11, R12, R16, R17, R2, R21, R22, R26, R27, R31, R32, R36, R37, R41, R42, R46, R47, R51, R52, R56, R57, R6, R61, R62, R66, R67, R7, R71, R72, R76, R77: footprint YoshLibrary:R_Axial_DIN0207_L6.3mm_D2.5mm_P7.62mm_Horizontal_Y -> Resistor_THT:R_Axial_DIN0207_L6.3mm_D2.5mm_P7.62mm_Horizontal
- R10, R15, R20, R25, R30, R35, R40, R45, R5, R50, R55, R60, R65, R70, R75, R80: value 5.1k -> 10k; footprint YoshLibrary:R_Axial_DIN0207_L6.3mm_D2.5mm_P7.62mm_Horizontal_Y -> Resistor_THT:R_Axial_DIN0207_L6.3mm_D2.5mm_P7.62mm_Horizontal
- R13, R18, R23, R28, R3, R33, R38, R43, R48, R53, R58, R63, R68, R73, R78, R8: value 1k -> 5.1k; footprint YoshLibrary:R_Axial_DIN0207_L6.3mm_D2.5mm_P7.62mm_Horizontal_Y -> Resistor_THT:R_Axial_DIN0207_L6.3mm_D2.5mm_P7.62mm_Horizontal
- R14, R19, R24, R29, R34, R39, R4, R44, R49, R54, R59, R64, R69, R74, R79, R9: value 10k -> 5.1k; footprint YoshLibrary:R_Axial_DIN0207_L6.3mm_D2.5mm_P7.62mm_Horizontal_Y -> Resistor_THT:R_Axial_DIN0207_L6.3mm_D2.5mm_P7.62mm_Horizontal
- moved J1 328.7 mm to (377.9, 132.1), turned to 0 degrees
- moved D37 318.7 mm to (364.4, 75.5), turned to 0 degrees
- moved PQ25 317.6 mm to (365.4, 65.4), turned to 0 degrees
- moved D38 317.4 mm to (364.4, 79.0), turned to 0 degrees
- moved NQ85 313.6 mm to (345.9, 65.4)
- moved J2 313.1 mm to (382.5, 132.1), turned to 0 degrees
- moved NQ87 312.4 mm to (356.2, 77.0), turned to 0 degrees
- moved C13 312.3 mm to (364.4, 86.1)
- moved PX13 310.5 mm to (365.4, 71.2)
- moved R61 308.7 mm to (345.5, 75.7), turned to 0 degrees
- moved D39 307.3 mm to (364.4, 82.6), turned to 0 degrees
- moved NQ88 300.8 mm to (352.4, 65.4), turned to 0 degrees
- moved NQ89 300.6 mm to (352.4, 71.2), turned to 0 degrees
- moved J3 300.0 mm to (387.1, 132.1), turned to 0 degrees
- moved NQ86 299.3 mm to (345.9, 71.2), turned to 0 degrees
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Connections:
- C1 pad 2: Net-(D3-A) -> Net-(D1-A)
- C10 pad 2: Net-(D30-A) -> Net-(D28-A)
- C11 pad 2: Net-(D33-A) -> Net-(D31-A)
- C12 pad 2: Net-(D36-A) -> Net-(D34-A)
- C13 pad 2: Net-(D39-A) -> Net-(D37-A)
- C14 pad 2: Net-(D42-A) -> Net-(D40-A)
- C15 pad 2: Net-(D45-A) -> Net-(D43-A)
- C16 pad 2: Net-(D48-A) -> Net-(D46-A)
- C2 pad 2: Net-(D6-A) -> Net-(D4-A)
- C3 pad 2: Net-(D9-A) -> Net-(D7-A)
- C4 pad 2: Net-(D12-A) -> Net-(D10-A)
- C5 pad 2: Net-(D15-A) -> Net-(D13-A)
- C6 pad 2: Net-(D18-A) -> Net-(D16-A)
- C7 pad 2: Net-(D21-A) -> Net-(D19-A)
- C8 pad 2: Net-(D24-A) -> Net-(D22-A)
- C9 pad 2: Net-(D27-A) -> Net-(D25-A)
- D1 pad 2: /Rst -> Net-(D1-A)
- D10 pad 2: /Rst -> Net-(D10-A)
- D11 pad 1: Net-(D10-K) -> Net-(D11-K)
- D12 pad 1: Net-(D12-K) -> Net-(D11-K)
- D12 pad 2: Net-(D12-A) -> /Rst
- D13 pad 2: /Rst -> Net-(D13-A)
- D14 pad 1: Net-(D13-K) -> Net-(D14-K)
- D15 pad 1: Net-(D15-K) -> Net-(D14-K)
- D15 pad 2: Net-(D15-A) -> /Rst
- D16 pad 2: /Rst -> Net-(D16-A)
- D17 pad 1: Net-(D16-K) -> Net-(D17-K)
- D18 pad 1: Net-(D18-K) -> Net-(D17-K)
- D18 pad 2: Net-(D18-A) -> /Rst
- D19 pad 2: /Rst -> Net-(D19-A)
- D2 pad 1: Net-(D1-K) -> Net-(D2-K)
- D20 pad 1: Net-(D19-K) -> Net-(D20-K)
- D21 pad 1: Net-(D21-K) -> Net-(D20-K)
- D21 pad 2: Net-(D21-A) -> /Rst
- D22 pad 2: /Rst -> Net-(D22-A)
- D23 pad 1: Net-(D22-K) -> Net-(D23-K)
- D24 pad 1: Net-(D24-K) -> Net-(D23-K)
- D24 pad 2: Net-(D24-A) -> /Rst
- D25 pad 2: /Rst -> Net-(D25-A)
- D26 pad 1: Net-(D25-K) -> Net-(D26-K)
- D27 pad 1: Net-(D27-K) -> Net-(D26-K)
- D27 pad 2: Net-(D27-A) -> /Rst
- D28 pad 2: /Rst -> Net-(D28-A)
- D29 pad 1: Net-(D28-K) -> Net-(D29-K)
- D3 pad 1: Net-(D3-K) -> Net-(D2-K)
- D3 pad 2: Net-(D3-A) -> /Rst
- D30 pad 1: Net-(D30-K) -> Net-(D29-K)
- D30 pad 2: Net-(D30-A) -> /Rst
- D31 pad 2: /Rst -> Net-(D31-A)
- D32 pad 1: Net-(D31-K) -> Net-(D32-K)
- D33 pad 1: Net-(D33-K) -> Net-(D32-K)
- D33 pad 2: Net-(D33-A) -> /Rst
- D34 pad 2: /Rst -> Net-(D34-A)
- D35 pad 1: Net-(D34-K) -> Net-(D35-K)
- D36 pad 1: Net-(D36-K) -> Net-(D35-K)
- D36 pad 2: Net-(D36-A) -> /Rst
- D37 pad 2: /Rst -> Net-(D37-A)
- D38 pad 1: Net-(D37-K) -> Net-(D38-K)
- D39 pad 1: Net-(D39-K) -> Net-(D38-K)
- D39 pad 2: Net-(D39-A) -> /Rst
- D4 pad 2: /Rst -> Net-(D4-A)
- D40 pad 2: /Rst -> Net-(D40-A)
- D41 pad 1: Net-(D40-K) -> Net-(D41-K)
- D42 pad 1: Net-(D42-K) -> Net-(D41-K)
- D42 pad 2: Net-(D42-A) -> /Rst
- D43 pad 2: /Rst -> Net-(D43-A)
- D44 pad 1: Net-(D43-K) -> Net-(D44-K)
- D45 pad 1: Net-(D45-K) -> Net-(D44-K)
- D45 pad 2: Net-(D45-A) -> /Rst
- D46 pad 2: /Rst -> Net-(D46-A)
- D47 pad 1: Net-(D46-K) -> Net-(D47-K)
- D48 pad 1: Net-(D48-K) -> Net-(D47-K)
- D48 pad 2: Net-(D48-A) -> /Rst
- D5 pad 1: Net-(D4-K) -> Net-(D5-K)
- D6 pad 1: Net-(D6-K) -> Net-(D5-K)
- D6 pad 2: Net-(D6-A) -> /Rst
- D7 pad 2: /Rst -> Net-(D7-A)
- D8 pad 1: Net-(D7-K) -> Net-(D8-K)
- D9 pad 1: Net-(D9-K) -> Net-(D8-K)
- D9 pad 2: Net-(D9-A) -> /Rst
- NQ1 pad 1: GND -> Net-(NQ1-E)
- NQ1 pad 2: Net-(D2-A) -> Net-(NQ1-C)
- NQ1 pad 3: /D0 -> /WEn
- NQ10 pad 3: /WEn -> /DEn
- NQ101 pad 1: Net-(NQ100-C) -> Net-(NQ101-E)
- NQ101 pad 3: /WEn -> /DEn
- NQ102 pad 2: Net-(D45-K) -> Net-(D43-K)
- NQ102 pad 3: Net-(D43-K) -> Net-(D44-K)
- NQ103 pad 2: Net-(NQ102-E) -> Net-(D44-A)
- NQ103 pad 3: /WEn -> /D14
- NQ104 pad 2: Net-(NQ104-C) -> Net-(NQ102-E)
- NQ104 pad 3: Net-(NQ104-B) -> /Rst
- NQ105 pad 1: Net-(NQ104-C) -> GND
- NQ105 pad 2: Net-(NQ105-C) -> Net-(NQ101-E)
- NQ105 pad 3: /DEn -> Net-(NQ105-B)
- NQ106 pad 1: GND -> Net-(NQ106-E)
- NQ106 pad 2: Net-(D47-A) -> Net-(NQ106-C)
- NQ106 pad 3: /D15 -> /WEn
- NQ107 pad 2: Net-(NQ107-C) -> Net-(NQ106-E)
- NQ108 pad 1: Net-(NQ107-C) -> Net-(NQ108-E)
- NQ108 pad 3: /WEn -> /DEn
- NQ109 pad 2: Net-(D48-K) -> Net-(D46-K)
- NQ109 pad 3: Net-(D46-K) -> Net-(D47-K)
- NQ11 pad 2: Net-(D6-K) -> Net-(D4-K)
- NQ11 pad 3: Net-(D4-K) -> Net-(D5-K)
- NQ110 pad 2: Net-(NQ109-E) -> Net-(D47-A)
- NQ110 pad 3: /WEn -> /D15
- NQ111 pad 2: Net-(NQ111-C) -> Net-(NQ109-E)
- NQ111 pad 3: Net-(NQ111-B) -> /Rst
- NQ112 pad 1: Net-(NQ111-C) -> GND
- NQ112 pad 2: Net-(NQ112-C) -> Net-(NQ108-E)
- NQ112 pad 3: /DEn -> Net-(NQ112-B)
- NQ12 pad 2: Net-(NQ11-E) -> Net-(D5-A)
- NQ12 pad 3: /WEn -> /D1
- NQ13 pad 2: Net-(NQ13-C) -> Net-(NQ11-E)
- NQ13 pad 3: Net-(NQ13-B) -> /Rst
- NQ14 pad 1: Net-(NQ13-C) -> GND
- NQ14 pad 2: Net-(NQ14-C) -> Net-(NQ10-E)
- NQ14 pad 3: /DEn -> Net-(NQ14-B)
- NQ15 pad 1: GND -> Net-(NQ15-E)
- NQ15 pad 2: Net-(D8-A) -> Net-(NQ15-C)
- NQ15 pad 3: /D2 -> /WEn
- NQ16 pad 2: Net-(NQ16-C) -> Net-(NQ15-E)
- NQ17 pad 1: Net-(NQ16-C) -> Net-(NQ17-E)
- NQ17 pad 3: /WEn -> /DEn
- NQ18 pad 2: Net-(D9-K) -> Net-(D7-K)
- NQ18 pad 3: Net-(D7-K) -> Net-(D8-K)
- NQ19 pad 2: Net-(NQ18-E) -> Net-(D8-A)
- NQ19 pad 3: /WEn -> /D2
- NQ2 pad 2: Net-(NQ2-C) -> Net-(NQ1-E)
- NQ20 pad 2: Net-(NQ20-C) -> Net-(NQ18-E)
- NQ20 pad 3: Net-(NQ20-B) -> /Rst
- NQ21 pad 1: Net-(NQ20-C) -> GND
- NQ21 pad 2: Net-(NQ21-C) -> Net-(NQ17-E)
- NQ21 pad 3: /DEn -> Net-(NQ21-B)
- NQ22 pad 1: GND -> Net-(NQ22-E)
- NQ22 pad 2: Net-(D11-A) -> Net-(NQ22-C)
- NQ22 pad 3: /D3 -> /WEn
- NQ23 pad 2: Net-(NQ23-C) -> Net-(NQ22-E)
- NQ24 pad 1: Net-(NQ23-C) -> Net-(NQ24-E)
- NQ24 pad 3: /WEn -> /DEn
- NQ25 pad 2: Net-(D12-K) -> Net-(D10-K)
- NQ25 pad 3: Net-(D10-K) -> Net-(D11-K)
- NQ26 pad 2: Net-(NQ25-E) -> Net-(D11-A)
- NQ26 pad 3: /WEn -> /D3
- NQ27 pad 2: Net-(NQ27-C) -> Net-(NQ25-E)
- NQ27 pad 3: Net-(NQ27-B) -> /Rst
- NQ28 pad 1: Net-(NQ27-C) -> GND
- NQ28 pad 2: Net-(NQ28-C) -> Net-(NQ24-E)
- NQ28 pad 3: /DEn -> Net-(NQ28-B)
- NQ29 pad 1: GND -> Net-(NQ29-E)
- NQ29 pad 2: Net-(D14-A) -> Net-(NQ29-C)
- NQ29 pad 3: /D4 -> /WEn
- NQ3 pad 1: Net-(NQ2-C) -> Net-(NQ3-E)
- NQ3 pad 3: /WEn -> /DEn
- NQ30 pad 2: Net-(NQ30-C) -> Net-(NQ29-E)
- NQ31 pad 1: Net-(NQ30-C) -> Net-(NQ31-E)
- NQ31 pad 3: /WEn -> /DEn
- NQ32 pad 2: Net-(D15-K) -> Net-(D13-K)
- NQ32 pad 3: Net-(D13-K) -> Net-(D14-K)
- NQ33 pad 2: Net-(NQ32-E) -> Net-(D14-A)
- NQ33 pad 3: /WEn -> /D4
- NQ34 pad 2: Net-(NQ34-C) -> Net-(NQ32-E)
- NQ34 pad 3: Net-(NQ34-B) -> /Rst
- NQ35 pad 1: Net-(NQ34-C) -> GND
- NQ35 pad 2: Net-(NQ35-C) -> Net-(NQ31-E)
- NQ35 pad 3: /DEn -> Net-(NQ35-B)
- NQ36 pad 1: GND -> Net-(NQ36-E)
- NQ36 pad 2: Net-(D17-A) -> Net-(NQ36-C)
- NQ36 pad 3: /D5 -> /WEn
- NQ37 pad 2: Net-(NQ37-C) -> Net-(NQ36-E)
- NQ38 pad 1: Net-(NQ37-C) -> Net-(NQ38-E)
- NQ38 pad 3: /WEn -> /DEn
- NQ39 pad 2: Net-(D18-K) -> Net-(D16-K)
- NQ39 pad 3: Net-(D16-K) -> Net-(D17-K)
- NQ4 pad 2: Net-(D3-K) -> Net-(D1-K)
- NQ4 pad 3: Net-(D1-K) -> Net-(D2-K)
- NQ40 pad 2: Net-(NQ39-E) -> Net-(D17-A)
- NQ40 pad 3: /WEn -> /D5
- NQ41 pad 2: Net-(NQ41-C) -> Net-(NQ39-E)
- NQ41 pad 3: Net-(NQ41-B) -> /Rst
- NQ42 pad 1: Net-(NQ41-C) -> GND
- NQ42 pad 2: Net-(NQ42-C) -> Net-(NQ38-E)
- NQ42 pad 3: /DEn -> Net-(NQ42-B)
- NQ43 pad 1: GND -> Net-(NQ43-E)
- NQ43 pad 2: Net-(D20-A) -> Net-(NQ43-C)
- NQ43 pad 3: /D6 -> /WEn
- NQ44 pad 2: Net-(NQ44-C) -> Net-(NQ43-E)
- NQ45 pad 1: Net-(NQ44-C) -> Net-(NQ45-E)
- NQ45 pad 3: /WEn -> /DEn
- NQ46 pad 2: Net-(D21-K) -> Net-(D19-K)
- NQ46 pad 3: Net-(D19-K) -> Net-(D20-K)
- NQ47 pad 2: Net-(NQ46-E) -> Net-(D20-A)
- NQ47 pad 3: /WEn -> /D6
- NQ48 pad 2: Net-(NQ48-C) -> Net-(NQ46-E)
- NQ48 pad 3: Net-(NQ48-B) -> /Rst
- NQ49 pad 1: Net-(NQ48-C) -> GND
- NQ49 pad 2: Net-(NQ49-C) -> Net-(NQ45-E)
- NQ49 pad 3: /DEn -> Net-(NQ49-B)
- NQ5 pad 2: Net-(NQ4-E) -> Net-(D2-A)
- NQ5 pad 3: /WEn -> /D0
- NQ50 pad 1: GND -> Net-(NQ50-E)
- NQ50 pad 2: Net-(D23-A) -> Net-(NQ50-C)
- NQ50 pad 3: /D7 -> /WEn
- NQ51 pad 2: Net-(NQ51-C) -> Net-(NQ50-E)
- NQ52 pad 1: Net-(NQ51-C) -> Net-(NQ52-E)
- NQ52 pad 3: /WEn -> /DEn
- NQ53 pad 2: Net-(D24-K) -> Net-(D22-K)
- NQ53 pad 3: Net-(D22-K) -> Net-(D23-K)
- NQ54 pad 2: Net-(NQ53-E) -> Net-(D23-A)
- NQ54 pad 3: /WEn -> /D7
- NQ55 pad 2: Net-(NQ55-C) -> Net-(NQ53-E)
- NQ55 pad 3: Net-(NQ55-B) -> /Rst
- NQ56 pad 1: Net-(NQ55-C) -> GND
- NQ56 pad 2: Net-(NQ56-C) -> Net-(NQ52-E)
- NQ56 pad 3: /DEn -> Net-(NQ56-B)
- NQ57 pad 1: GND -> Net-(NQ57-E)
- NQ57 pad 2: Net-(D26-A) -> Net-(NQ57-C)
- NQ57 pad 3: /D8 -> /WEn
- NQ58 pad 2: Net-(NQ58-C) -> Net-(NQ57-E)
- NQ59 pad 1: Net-(NQ58-C) -> Net-(NQ59-E)
- NQ59 pad 3: /WEn -> /DEn
- NQ6 pad 2: Net-(NQ6-C) -> Net-(NQ4-E)
- NQ6 pad 3: Net-(NQ6-B) -> /Rst
- NQ60 pad 2: Net-(D27-K) -> Net-(D25-K)
- NQ60 pad 3: Net-(D25-K) -> Net-(D26-K)
- NQ61 pad 2: Net-(NQ60-E) -> Net-(D26-A)
- NQ61 pad 3: /WEn -> /D8
- NQ62 pad 2: Net-(NQ62-C) -> Net-(NQ60-E)
- NQ62 pad 3: Net-(NQ62-B) -> /Rst
- NQ63 pad 1: Net-(NQ62-C) -> GND
- NQ63 pad 2: Net-(NQ63-C) -> Net-(NQ59-E)
- NQ63 pad 3: /DEn -> Net-(NQ63-B)
- NQ64 pad 1: GND -> Net-(NQ64-E)
- NQ64 pad 2: Net-(D29-A) -> Net-(NQ64-C)
- NQ64 pad 3: /D9 -> /WEn
- NQ65 pad 2: Net-(NQ65-C) -> Net-(NQ64-E)
- NQ66 pad 1: Net-(NQ65-C) -> Net-(NQ66-E)
- NQ66 pad 3: /WEn -> /DEn
- NQ67 pad 2: Net-(D30-K) -> Net-(D28-K)
- NQ67 pad 3: Net-(D28-K) -> Net-(D29-K)
- NQ68 pad 2: Net-(NQ67-E) -> Net-(D29-A)
- NQ68 pad 3: /WEn -> /D9
- NQ69 pad 2: Net-(NQ69-C) -> Net-(NQ67-E)
- NQ69 pad 3: Net-(NQ69-B) -> /Rst
- NQ7 pad 1: Net-(NQ6-C) -> GND
- NQ7 pad 2: Net-(NQ7-C) -> Net-(NQ3-E)
- NQ7 pad 3: /DEn -> Net-(NQ7-B)
- NQ70 pad 1: Net-(NQ69-C) -> GND
- NQ70 pad 2: Net-(NQ70-C) -> Net-(NQ66-E)
- NQ70 pad 3: /DEn -> Net-(NQ70-B)
- NQ71 pad 1: GND -> Net-(NQ71-E)
- NQ71 pad 2: Net-(D32-A) -> Net-(NQ71-C)
- NQ71 pad 3: /D10 -> /WEn
- NQ72 pad 2: Net-(NQ72-C) -> Net-(NQ71-E)
- NQ73 pad 1: Net-(NQ72-C) -> Net-(NQ73-E)
- NQ73 pad 3: /WEn -> /DEn
- NQ74 pad 2: Net-(D33-K) -> Net-(D31-K)
- NQ74 pad 3: Net-(D31-K) -> Net-(D32-K)
- NQ75 pad 2: Net-(NQ74-E) -> Net-(D32-A)
- NQ75 pad 3: /WEn -> /D10
- NQ76 pad 2: Net-(NQ76-C) -> Net-(NQ74-E)
- NQ76 pad 3: Net-(NQ76-B) -> /Rst
- NQ77 pad 1: Net-(NQ76-C) -> GND
- NQ77 pad 2: Net-(NQ77-C) -> Net-(NQ73-E)
- NQ77 pad 3: /DEn -> Net-(NQ77-B)
- NQ78 pad 1: GND -> Net-(NQ78-E)
- NQ78 pad 2: Net-(D35-A) -> Net-(NQ78-C)
- NQ78 pad 3: /D11 -> /WEn
- NQ79 pad 2: Net-(NQ79-C) -> Net-(NQ78-E)
- NQ8 pad 1: GND -> Net-(NQ8-E)
- NQ8 pad 2: Net-(D5-A) -> Net-(NQ8-C)
- NQ8 pad 3: /D1 -> /WEn
- NQ80 pad 1: Net-(NQ79-C) -> Net-(NQ80-E)
- NQ80 pad 3: /WEn -> /DEn
- NQ81 pad 2: Net-(D36-K) -> Net-(D34-K)
- NQ81 pad 3: Net-(D34-K) -> Net-(D35-K)
- NQ82 pad 2: Net-(NQ81-E) -> Net-(D35-A)
- NQ82 pad 3: /WEn -> /D11
- NQ83 pad 2: Net-(NQ83-C) -> Net-(NQ81-E)
- NQ83 pad 3: Net-(NQ83-B) -> /Rst
- NQ84 pad 1: Net-(NQ83-C) -> GND
- NQ84 pad 2: Net-(NQ84-C) -> Net-(NQ80-E)
- NQ84 pad 3: /DEn -> Net-(NQ84-B)
- NQ85 pad 1: GND -> Net-(NQ85-E)
- NQ85 pad 2: Net-(D38-A) -> Net-(NQ85-C)
- NQ85 pad 3: /D12 -> /WEn
- NQ86 pad 2: Net-(NQ86-C) -> Net-(NQ85-E)
- NQ87 pad 1: Net-(NQ86-C) -> Net-(NQ87-E)
- NQ87 pad 3: /WEn -> /DEn
- NQ88 pad 2: Net-(D39-K) -> Net-(D37-K)
- NQ88 pad 3: Net-(D37-K) -> Net-(D38-K)
- NQ89 pad 2: Net-(NQ88-E) -> Net-(D38-A)
- NQ89 pad 3: /WEn -> /D12
- NQ9 pad 2: Net-(NQ10-E) -> Net-(NQ8-E)
- NQ90 pad 2: Net-(NQ90-C) -> Net-(NQ88-E)
- NQ90 pad 3: Net-(NQ90-B) -> /Rst
- NQ91 pad 1: Net-(NQ90-C) -> GND
- NQ91 pad 2: Net-(NQ91-C) -> Net-(NQ87-E)
- NQ91 pad 3: /DEn -> Net-(NQ91-B)
- NQ92 pad 1: GND -> Net-(NQ92-E)
- NQ92 pad 2: Net-(D41-A) -> Net-(NQ92-C)
- NQ92 pad 3: /D13 -> /WEn
- NQ93 pad 2: Net-(NQ93-C) -> Net-(NQ92-E)
- NQ94 pad 1: Net-(NQ93-C) -> Net-(NQ94-E)
- NQ94 pad 3: /WEn -> /DEn
- NQ95 pad 2: Net-(D42-K) -> Net-(D40-K)
- NQ95 pad 3: Net-(D40-K) -> Net-(D41-K)
- NQ96 pad 2: Net-(NQ95-E) -> Net-(D41-A)
- NQ96 pad 3: /WEn -> /D13
- NQ97 pad 2: Net-(NQ97-C) -> Net-(NQ95-E)
- NQ97 pad 3: Net-(NQ97-B) -> /Rst
- NQ98 pad 1: Net-(NQ97-C) -> GND
- NQ98 pad 2: Net-(NQ98-C) -> Net-(NQ94-E)
- NQ98 pad 3: /DEn -> Net-(NQ98-B)
- NQ99 pad 1: GND -> Net-(NQ100-C)
- NQ99 pad 2: Net-(D44-A) -> Net-(NQ99-C)
- NQ99 pad 3: /D14 -> /WEn
- NX1 pad 1: Net-(NQ6-B) -> Net-(NQ7-B)
- NX1 pad 3: Net-(D3-A) -> Net-(D1-A)
- NX10 pad 1: Net-(NQ69-B) -> Net-(NQ70-B)
- NX10 pad 3: Net-(D30-A) -> Net-(D28-A)
- NX11 pad 1: Net-(NQ76-B) -> Net-(NQ77-B)
- NX11 pad 3: Net-(D33-A) -> Net-(D31-A)
- NX12 pad 1: Net-(NQ83-B) -> Net-(NQ84-B)
- NX12 pad 3: Net-(D36-A) -> Net-(D34-A)
- NX13 pad 1: Net-(NQ90-B) -> Net-(NQ91-B)
- NX13 pad 3: Net-(D39-A) -> Net-(D37-A)
- NX14 pad 1: Net-(NQ97-B) -> Net-(NQ98-B)
- NX14 pad 3: Net-(D42-A) -> Net-(D40-A)
- NX15 pad 1: Net-(NQ104-B) -> Net-(NQ105-B)
- NX15 pad 3: Net-(D45-A) -> Net-(D43-A)
- NX16 pad 1: Net-(NQ111-B) -> Net-(NQ112-B)
- NX16 pad 3: Net-(D48-A) -> Net-(D46-A)
- NX2 pad 1: Net-(NQ13-B) -> Net-(NQ14-B)
- NX2 pad 3: Net-(D6-A) -> Net-(D4-A)
- NX3 pad 1: Net-(NQ20-B) -> Net-(NQ21-B)
- NX3 pad 3: Net-(D9-A) -> Net-(D7-A)
- NX4 pad 1: Net-(NQ27-B) -> Net-(NQ28-B)
- NX4 pad 3: Net-(D12-A) -> Net-(D10-A)
- NX5 pad 1: Net-(NQ34-B) -> Net-(NQ35-B)
- NX5 pad 3: Net-(D15-A) -> Net-(D13-A)
- NX6 pad 1: Net-(NQ41-B) -> Net-(NQ42-B)
- NX6 pad 3: Net-(D18-A) -> Net-(D16-A)
- NX7 pad 1: Net-(NQ48-B) -> Net-(NQ49-B)
- NX7 pad 3: Net-(D21-A) -> Net-(D19-A)
- NX8 pad 1: Net-(NQ55-B) -> Net-(NQ56-B)
- NX8 pad 3: Net-(D24-A) -> Net-(D22-A)
- NX9 pad 1: Net-(NQ62-B) -> Net-(NQ63-B)
- NX9 pad 3: Net-(D27-A) -> Net-(D25-A)
- PQ1 pad 3: Net-(NQ3-C) -> Net-(NQ1-C)
- PQ10 pad 3: Net-(NQ35-C) -> Net-(NQ31-C)
- PQ11 pad 3: Net-(NQ38-C) -> Net-(NQ36-C)
- PQ12 pad 3: Net-(NQ42-C) -> Net-(NQ38-C)
- PQ13 pad 3: Net-(NQ45-C) -> Net-(NQ43-C)
- PQ14 pad 3: Net-(NQ49-C) -> Net-(NQ45-C)
- PQ15 pad 3: Net-(NQ52-C) -> Net-(NQ50-C)
- PQ16 pad 3: Net-(NQ56-C) -> Net-(NQ52-C)
- PQ17 pad 3: Net-(NQ59-C) -> Net-(NQ57-C)
- PQ18 pad 3: Net-(NQ63-C) -> Net-(NQ59-C)
- PQ19 pad 3: Net-(NQ66-C) -> Net-(NQ64-C)
- PQ2 pad 3: Net-(NQ7-C) -> Net-(NQ3-C)
- PQ20 pad 3: Net-(NQ70-C) -> Net-(NQ66-C)
- PQ21 pad 3: Net-(NQ73-C) -> Net-(NQ71-C)
- PQ22 pad 3: Net-(NQ77-C) -> Net-(NQ73-C)
- PQ23 pad 3: Net-(NQ80-C) -> Net-(NQ78-C)
- PQ24 pad 3: Net-(NQ84-C) -> Net-(NQ80-C)
- PQ25 pad 3: Net-(NQ87-C) -> Net-(NQ85-C)
- PQ26 pad 3: Net-(NQ91-C) -> Net-(NQ87-C)
- PQ27 pad 3: Net-(NQ94-C) -> Net-(NQ92-C)
- PQ28 pad 3: Net-(NQ98-C) -> Net-(NQ94-C)
- PQ29 pad 3: Net-(NQ101-C) -> Net-(NQ99-C)
- PQ3 pad 3: Net-(NQ10-C) -> Net-(NQ8-C)
- PQ30 pad 3: Net-(NQ105-C) -> Net-(NQ101-C)
- PQ31 pad 3: Net-(NQ108-C) -> Net-(NQ106-C)
- PQ32 pad 3: Net-(NQ112-C) -> Net-(NQ108-C)
- PQ4 pad 3: Net-(NQ14-C) -> Net-(NQ10-C)
- PQ5 pad 3: Net-(NQ17-C) -> Net-(NQ15-C)
- PQ6 pad 3: Net-(NQ21-C) -> Net-(NQ17-C)
- PQ7 pad 3: Net-(NQ24-C) -> Net-(NQ22-C)
- PQ8 pad 3: Net-(NQ28-C) -> Net-(NQ24-C)
- PQ9 pad 3: Net-(NQ31-C) -> Net-(NQ29-C)
- PX1 pad 2: Net-(D3-A) -> Net-(D1-A)
- PX10 pad 2: Net-(D30-A) -> Net-(D28-A)
- PX11 pad 2: Net-(D33-A) -> Net-(D31-A)
- PX12 pad 2: Net-(D36-A) -> Net-(D34-A)
- PX13 pad 2: Net-(D39-A) -> Net-(D37-A)
- PX14 pad 2: Net-(D42-A) -> Net-(D40-A)
- PX15 pad 2: Net-(D45-A) -> Net-(D43-A)
- PX16 pad 2: Net-(D48-A) -> Net-(D46-A)
- PX2 pad 2: Net-(D6-A) -> Net-(D4-A)
- PX3 pad 2: Net-(D9-A) -> Net-(D7-A)
- PX4 pad 2: Net-(D12-A) -> Net-(D10-A)
- PX5 pad 2: Net-(D15-A) -> Net-(D13-A)
- PX6 pad 2: Net-(D18-A) -> Net-(D16-A)
- PX7 pad 2: Net-(D21-A) -> Net-(D19-A)
- PX8 pad 2: Net-(D24-A) -> Net-(D22-A)
- PX9 pad 2: Net-(D27-A) -> Net-(D25-A)
- R1 pad 1: /WEn -> Net-(PX1-E)
- R1 pad 2: Net-(D2-A) -> +5V
- R10 pad 1: Net-(NX2-C) -> Net-(D4-A)
- R10 pad 2: Net-(PX2-E) -> GND
- R11 pad 1: /WEn -> Net-(PX3-E)
- R11 pad 2: Net-(D8-A) -> +5V
- R12 pad 1: Net-(D9-A) -> Net-(D8-A)
- R12 pad 2: Net-(PQ5-C) -> /WEn
- R13 pad 1: Net-(PX3-E) -> Net-(NX3-C)
- R13 pad 2: +5V -> Net-(PX3-E)
- R14 pad 1: Net-(D9-A) -> Net-(D7-A)
- R14 pad 2: GND -> Net-(PQ5-C)
- R15 pad 1: Net-(NX3-C) -> Net-(D7-A)
- R15 pad 2: Net-(PX3-E) -> GND
- R16 pad 1: /WEn -> Net-(PX4-E)
- R16 pad 2: Net-(D11-A) -> +5V
- R17 pad 1: Net-(D12-A) -> Net-(D11-A)
- R17 pad 2: Net-(PQ7-C) -> /WEn
- R18 pad 1: Net-(PX4-E) -> Net-(NX4-C)
- R18 pad 2: +5V -> Net-(PX4-E)
- R19 pad 1: Net-(D12-A) -> Net-(D10-A)
- R19 pad 2: GND -> Net-(PQ7-C)
- R2 pad 1: Net-(D3-A) -> Net-(D2-A)
- R2 pad 2: Net-(PQ1-C) -> /WEn
- R20 pad 1: Net-(NX4-C) -> Net-(D10-A)
- R20 pad 2: Net-(PX4-E) -> GND
- R21 pad 1: /WEn -> Net-(PX5-E)
- R21 pad 2: Net-(D14-A) -> +5V
- R22 pad 1: Net-(D15-A) -> Net-(D14-A)
- R22 pad 2: Net-(PQ9-C) -> /WEn
- R23 pad 1: Net-(PX5-E) -> Net-(NX5-C)
- R23 pad 2: +5V -> Net-(PX5-E)
- R24 pad 1: Net-(D15-A) -> Net-(D13-A)
- R24 pad 2: GND -> Net-(PQ9-C)
- R25 pad 1: Net-(NX5-C) -> Net-(D13-A)
- R25 pad 2: Net-(PX5-E) -> GND
- R26 pad 1: /WEn -> Net-(PX6-E)
- R26 pad 2: Net-(D17-A) -> +5V
- R27 pad 1: Net-(D18-A) -> Net-(D17-A)
- R27 pad 2: Net-(PQ11-C) -> /WEn
- R28 pad 1: Net-(PX6-E) -> Net-(NX6-C)
- R28 pad 2: +5V -> Net-(PX6-E)
- R29 pad 1: Net-(D18-A) -> Net-(D16-A)
- R29 pad 2: GND -> Net-(PQ11-C)
- R3 pad 1: Net-(PX1-E) -> Net-(NX1-C)
- R3 pad 2: +5V -> Net-(PX1-E)
- R30 pad 1: Net-(NX6-C) -> Net-(D16-A)
- R30 pad 2: Net-(PX6-E) -> GND
- R31 pad 1: /WEn -> Net-(PX7-E)
- R31 pad 2: Net-(D20-A) -> +5V
- R32 pad 1: Net-(D21-A) -> Net-(D20-A)
- R32 pad 2: Net-(PQ13-C) -> /WEn
- R33 pad 1: Net-(PX7-E) -> Net-(NX7-C)
- R33 pad 2: +5V -> Net-(PX7-E)
- R34 pad 1: Net-(D21-A) -> Net-(D19-A)
- R34 pad 2: GND -> Net-(PQ13-C)
- R35 pad 1: Net-(NX7-C) -> Net-(D19-A)
- R35 pad 2: Net-(PX7-E) -> GND
- R36 pad 1: /WEn -> Net-(PX8-E)
- R36 pad 2: Net-(D23-A) -> +5V
- R37 pad 1: Net-(D24-A) -> Net-(D23-A)
- R37 pad 2: Net-(PQ15-C) -> /WEn
- R38 pad 1: Net-(PX8-E) -> Net-(NX8-C)
- R38 pad 2: +5V -> Net-(PX8-E)
- R39 pad 1: Net-(D24-A) -> Net-(D22-A)
- R39 pad 2: GND -> Net-(PQ15-C)
- R4 pad 1: Net-(D3-A) -> Net-(D1-A)
- R4 pad 2: GND -> Net-(PQ1-C)
- R40 pad 1: Net-(NX8-C) -> Net-(D22-A)
- R40 pad 2: Net-(PX8-E) -> GND
- R41 pad 1: /WEn -> Net-(PX9-E)
- R41 pad 2: Net-(D26-A) -> +5V
- R42 pad 1: Net-(D27-A) -> Net-(D26-A)
- R42 pad 2: Net-(PQ17-C) -> /WEn
- R43 pad 1: Net-(PX9-E) -> Net-(NX9-C)
- R43 pad 2: +5V -> Net-(PX9-E)
- R44 pad 1: Net-(D27-A) -> Net-(D25-A)
- R44 pad 2: GND -> Net-(PQ17-C)
- R45 pad 1: Net-(NX9-C) -> Net-(D25-A)
- R45 pad 2: Net-(PX9-E) -> GND
- R46 pad 1: /WEn -> Net-(PX10-E)
- R46 pad 2: Net-(D29-A) -> +5V
- R47 pad 1: Net-(D30-A) -> Net-(D29-A)
- R47 pad 2: Net-(PQ19-C) -> /WEn
- R48 pad 1: Net-(PX10-E) -> Net-(NX10-C)
- R48 pad 2: +5V -> Net-(PX10-E)
- R49 pad 1: Net-(D30-A) -> Net-(D28-A)
- R49 pad 2: GND -> Net-(PQ19-C)
- R5 pad 1: Net-(NX1-C) -> Net-(D1-A)
- R5 pad 2: Net-(PX1-E) -> GND
- R50 pad 1: Net-(NX10-C) -> Net-(D28-A)
- R50 pad 2: Net-(PX10-E) -> GND
- R51 pad 1: /WEn -> Net-(PX11-E)
- R51 pad 2: Net-(D32-A) -> +5V
- R52 pad 1: Net-(D33-A) -> Net-(D32-A)
- R52 pad 2: Net-(PQ21-C) -> /WEn
- R53 pad 1: Net-(PX11-E) -> Net-(NX11-C)
- R53 pad 2: +5V -> Net-(PX11-E)
- R54 pad 1: Net-(D33-A) -> Net-(D31-A)
- R54 pad 2: GND -> Net-(PQ21-C)
- R55 pad 1: Net-(NX11-C) -> Net-(D31-A)
- R55 pad 2: Net-(PX11-E) -> GND
- R56 pad 1: /WEn -> Net-(PX12-E)
- R56 pad 2: Net-(D35-A) -> +5V
- R57 pad 1: Net-(D36-A) -> Net-(D35-A)
- R57 pad 2: Net-(PQ23-C) -> /WEn
- R58 pad 1: Net-(PX12-E) -> Net-(NX12-C)
- R58 pad 2: +5V -> Net-(PX12-E)
- R59 pad 1: Net-(D36-A) -> Net-(D34-A)
- R59 pad 2: GND -> Net-(PQ23-C)
- R6 pad 1: /WEn -> Net-(PX2-E)
- R6 pad 2: Net-(D5-A) -> +5V
- R60 pad 1: Net-(NX12-C) -> Net-(D34-A)
- R60 pad 2: Net-(PX12-E) -> GND
- R61 pad 1: /WEn -> Net-(PX13-E)
- R61 pad 2: Net-(D38-A) -> +5V
- R62 pad 1: Net-(D39-A) -> Net-(D38-A)
- R62 pad 2: Net-(PQ25-C) -> /WEn
- R63 pad 1: Net-(PX13-E) -> Net-(NX13-C)
- R63 pad 2: +5V -> Net-(PX13-E)
- R64 pad 1: Net-(D39-A) -> Net-(D37-A)
- R64 pad 2: GND -> Net-(PQ25-C)
- R65 pad 1: Net-(NX13-C) -> Net-(D37-A)
- R65 pad 2: Net-(PX13-E) -> GND
- R66 pad 1: /WEn -> Net-(PX14-E)
- R66 pad 2: Net-(D41-A) -> +5V
- R67 pad 1: Net-(D42-A) -> Net-(D41-A)
- R67 pad 2: Net-(PQ27-C) -> /WEn
- R68 pad 1: Net-(PX14-E) -> Net-(NX14-C)
- R68 pad 2: +5V -> Net-(PX14-E)
- R69 pad 1: Net-(D42-A) -> Net-(D40-A)
- R69 pad 2: GND -> Net-(PQ27-C)
- R7 pad 1: Net-(D6-A) -> Net-(D5-A)
- R7 pad 2: Net-(PQ3-C) -> /WEn
- R70 pad 1: Net-(NX14-C) -> Net-(D40-A)
- R70 pad 2: Net-(PX14-E) -> GND
- R71 pad 1: /WEn -> Net-(PX15-E)
- R71 pad 2: Net-(D44-A) -> +5V
- R72 pad 1: Net-(D45-A) -> Net-(D44-A)
- R72 pad 2: Net-(PQ29-C) -> /WEn
- R73 pad 1: Net-(PX15-E) -> Net-(NX15-C)
- R73 pad 2: +5V -> Net-(PX15-E)
- R74 pad 1: Net-(D45-A) -> Net-(D43-A)
- R74 pad 2: GND -> Net-(PQ29-C)
- R75 pad 1: Net-(NX15-C) -> Net-(D43-A)
- R75 pad 2: Net-(PX15-E) -> GND
- R76 pad 1: /WEn -> Net-(PX16-E)
- R76 pad 2: Net-(D47-A) -> +5V
- R77 pad 1: Net-(D48-A) -> Net-(D47-A)
- R77 pad 2: Net-(PQ31-C) -> /WEn
- R78 pad 1: Net-(PX16-E) -> Net-(NX16-C)
- R78 pad 2: +5V -> Net-(PX16-E)
- R79 pad 1: Net-(D48-A) -> Net-(D46-A)
- R79 pad 2: GND -> Net-(PQ31-C)
- R8 pad 1: Net-(PX2-E) -> Net-(NX2-C)
- R8 pad 2: +5V -> Net-(PX2-E)
- R80 pad 1: Net-(NX16-C) -> Net-(D46-A)
- R80 pad 2: Net-(PX16-E) -> GND
- R9 pad 1: Net-(D6-A) -> Net-(D4-A)
- R9 pad 2: GND -> Net-(PQ3-C)
Routing:
- net GND: track 1616.1 -> 0.00 mm, vias 4 -> 0
- net +5V: track 833.1 -> 0.00 mm, vias 4 -> 0
- net /WEn: track 121.9 -> 0.00 mm
- net Net-(D42-A): track 25.4 -> 0.00 mm
- net Net-(D39-A): track 25.4 -> 0.00 mm
- net Net-(D30-A): track 25.4 -> 0.00 mm
- net Net-(D27-A): track 25.4 -> 0.00 mm
- net Net-(D6-A): track 25.4 -> 0.00 mm
- net Net-(D3-A): track 25.4 -> 0.00 mm
- net Net-(D18-A): track 25.4 -> 0.00 mm
- net Net-(D15-A): track 25.4 -> 0.00 mm
- net Net-(D48-A): track 25.4 -> 0.00 mm
- net Net-(D45-A): track 25.4 -> 0.00 mm
- net Net-(D36-A): track 25.4 -> 0.00 mm
- net Net-(D33-A): track 25.4 -> 0.00 mm
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Other:
- board outline removed
